File: pcb/KIA-OBD2-DISPLAY/KIA-OBD2-DISPLAY.kicad_sch (KiCad schematic)
At the start: 6 parts, among them U3 ESP32-C3-DevKitM-1, U4 CAP1188-1-CP-TR, U5 MCP2515-xSO, U6 TJA1050

Commit message: run update
Parts:
- removed U3: ESP32-C3-DevKitM-1, PCM_Espressif:ESP32-C3-DevKitM-1, symbol PCM_Espressif:ESP32-C3-DevKitM-1
- added U9: ESP32-C6-MINI-1/U, PCM_Espressif:ESP32-C6-MINI-1, symbol PCM_Espressif:ESP32-C6-MINI-1/U
Connections:
- net GND: now reaches U2.1 (GND)
- net GND: now also U1.1 (GND), U4.25 (GND), U5.9 (VSS), U6.2 (GND), U9.1 (GND), U9.11 (GND), U9.14 (GND), U9.2 (GND), U9.36 (GND), U9.37 (GND), U9.38 (GND), U9.39 (GND), U9.40 (GND), U9.41 (GND), U9.42 (GND), U9.43 (GND), U9.44 (GND), U9.45 (GND), U9.46 (GND), U9.47 (GND), U9.48 (GND), U9.49 (GND), U9.50 (GND), U9.51 (GND), U9.52 (GND), U9.53 (GND)
- net +3.3V: now reaches U2.2 (+5V)
- net +3.3V: now also U1.2 (+5V)
- net SCLK: now reaches U2.3 (SCLK)
- net SCLK: now also U1.3 (SCLK), U4.4 (SMCLK/BC_CLK/SPI_CLK), U5.13 (SCK), U9.15 (MTCK/GPIO6/ADC1_CH6)
- net MOSI: now reaches U2.4 (MOSI)
- net MOSI: now also U1.4 (MOSI), U4.2 (WAKE/SPI_MOSI), U5.14 (SI), U9.16 (MTDO/GPIO7)
- net REST: now reaches U2.5 (RES)
- net REST: now also U1.5 (RES), U9.24 (GPIO18)
- net DC: now reaches U2.6 (DC)
- net DC: now also U1.6 (DC), U9.23 (GPIO9)
- net CSD2: now reaches U2.7 (CS)
- net CSD2: now also U9.20 (GPIO15)
- net CSCAN: now reaches U4.1 (~{SPI_CS}#)
- net CSCAN: now also U5.16 (~{CS}), U9.25 (GPIO19), U9.26 (GPIO20)
- net MISO: now reaches U4.3 (SMDATA/SPI_MSIO/SPI_MISO)
- net MISO: now also U5.15 (SO), U9.10 (MTDI/GPIO5/ADC1_CH5)
- net at U6.1 (TXD): now also U5.2 (RXCAN)
- net at U6.4 (RXD): now also U5.1 (TXCAN)
- net CSD1: now reaches U1.7 (CS)
- net CSD1: now also U9.19 (GPIO14)
Other:
- moved on the sheet: U1, U2, U4, U5, U6

Commit message: pcb 3d work
Parts:
- removed U5: MCP2515-xSO, Package_SO:SOIC-18W_7.5x11.6mm_P1.27mm, symbol Interface_CAN_LIN:MCP2515-xSO
- added C1, C2, C3, C4: 22pF, symbol Device:C_Small
- added D1, D2, D3, D4, D5, D6, D7, D8: LED, symbol Device:LED
- added D9: D, symbol Device:D
- added JP1, JP2: VREF 3.3V, symbol Jumper:SolderJumper_2_Open
- added Q1: NPN, symbol Simulation_SPICE:NPN
- added R1, R10, R11, R12, R13, R2, R3, R4, R5, R6, R7, R8, R9: R, symbol Device:R
- added U10, U11: MCP2515-xST, Package_SO:TSSOP-20_4.4x6.5mm_P0.65mm, symbol Interface_CAN_LIN:MCP2515-xST
- added U7: TJA1050, TJA1050:SOT96-1, symbol TJA1050C:TJA1050
- added U8: ~, symbol D24V10F3:D24V10F3
- added Y1, Y2: Crystal, symbol Device:Crystal
- U1, U2: footprint (none) -> SH1122:SH1122
- U4: footprint CAP1188-1-CP-TR:QFN50P400X400X90-25N -> CAP1188:QFN50P400X400X90-25N
Connections:
- net +3.3V: now also U4.23 (VDD), U6.3 (VCC), U9.3 (3V3), D1.2 (A), D2.2 (A), D3.2 (A), D4.2 (A), D5.2 (A), D6.2 (A), D7.2 (A), D8.2 (A), JP1.1 (A), JP2.1 (A), R11.2, R2.1, U10.20 (VDD), U11.20 (VDD), U7.3 (VCC), U8. (VOUT)
- net CSCAN: now also U9.31 (U0TXD/GPIO16), U10.18 (~{CS}); no longer U4.1 (~{SPI_CS}#), U9.25 (GPIO19), U9.26 (GPIO20)
- net CSD1: now also U9.24 (GPIO18); no longer U9.19 (GPIO14)
- net CSD2: now also U9.25 (GPIO19); no longer U9.20 (GPIO15)
- net DC: now also U9.29 (GPIO23); no longer U9.23 (GPIO9)
- net GND: now also U4.14 (ADDR_COMM), U6.8 (S), C1.1, C2.1, C3.1, C4.1, Q1.3 (E), R13.2, U10.10 (VSS), U11.10 (VSS), U7.2 (GND), U7.8 (S), U8. (VOUT)
- net MISO: now also U9.5 (GPIO2/ADC1_CH2), U10.17 (SO), U11.17 (SO); no longer U9.10 (MTDI/GPIO5/ADC1_CH5)
- net MOSI: now also U10.16 (SI), U11.16 (SI)
- net REST: now also U9.28 (GPIO22), R1.2, R11.1, U10.19 (~{RESET}), U11.19 (~{RESET}); no longer U9.24 (GPIO18)
- net SCLK: now also U10.14 (SCK), U11.14 (SCK)
- net at U4.10 (LED6): now also R8.2
- net at U4.11 (LED7): now also R9.2
- net at U4.12 (LED8): now also R10.2
- net INTCAP: now reaches U4.13 (ALERT#)
- net INTCAP: now also U9.6 (GPIO3/ADC1_CH3)
- net NREST: now reaches U4.24 (RESET)
- net NREST: now also Q1.1 (C), R2.2
- net at U4.5 (LED1): now also R3.2
- net at U4.6 (LED2): now also R4.2
- net at U4.7 (LED3): now also R5.2
- net at U4.8 (LED4): now also R6.2
- net at U4.9 (LED5): now also R7.2
- net INTCAN2: now reaches U9.13 (GPIO1/ADC1_CH1/XTAL_32K_N)
- net INTCAN2: now also U11.13 (~{INT})
- net CSCAN2: now reaches U9.30 (U0RXD/GPIO17)
- net CSCAN2: now also U11.18 (~{CS})
- net INTCAN: now reaches U9.9 (MTMS/GPIO4/ADC1_CH4)
- net INTCAN: now also U10.13 (~{INT})
- net at U6.1 (TXD): now also U10.1 (TXCAN)
- net at U6.4 (RXD): now also U10.2 (RXCAN)
- net at U6.5 (VREF): now also JP1.2 (B)
- new net: C2.2, U10.9 (OSC1), Y1.1
- new net: D8.1 (K), R10.1
- new net: U11.1 (TXCAN), U7.1 (TXD)
- new net: U11.2 (RXCAN), U7.4 (RXD)
- new net: C3.2, U11.8 (OSC2), Y2.2
- new net: C4.2, U11.9 (OSC1), Y2.1
- new net: D5.1 (K), R7.1
- new net: JP2.2 (B), U7.5 (VREF)
- new net: D9.1 (K), R12.1
- new net: D2.1 (K), R4.1
- new net: D4.1 (K), R6.1
- new net: D7.1 (K), R9.1
- new net: Q1.2 (B), R1.1
- new net: D6.1 (K), R8.1
- new net: D1.1 (K), R3.1
- new net: D3.1 (K), R5.1
- new net: C1.2, U10.8 (OSC2), Y1.2
- new net +12V: U8. (VOUT)
- new net CSCAP: U4.1 (~{SPI_CS}#), U9.26 (GPIO20)
- new net ING12V+: D9.2 (A)
- new net INTING: R12.2, R13.1, U9.10 (MTDI/GPIO5/ADC1_CH5)
Other:
- moved on the sheet: U4, U6

Commit message: pcb update
Parts:
- removed JP1: VREF 3.3V, symbol Jumper:SolderJumper_2_Open
- removed Y1, Y2: Crystal, symbol Device:Crystal
- added F1: Fuse_Small, symbol Device:Fuse_Small
- added J1: Conn_01x07_Pin, Connector_PinHeader_2.54mm:PinHeader_1x07_P2.54mm_Horizontal, symbol Connector:Conn_01x07_Pin
- added Y1, Y4: Crystal_GND24_Small, Crystal:Crystal_SMD_3225-4Pin_3.2x2.5mm_HandSoldering, symbol Device:Crystal_GND24_Small
- JP2: footprint (none) -> Jumper:SolderJumper-2_P1.3mm_Open_RoundedPad1.0x1.5mm
- U8: footprint (none) -> D24V10F3:D24V10F3
Connections:
- net +12V: now also U8.3 (VIN), F1.1; no longer U8. (VOUT)
- net +3.3V: now also U8.1 (VOUT); no longer U8. (VOUT)
- net GND: now also C2.2, U10.9 (OSC1), U8.2 (GND), J1.2 (Pin_2), Y1.2, Y1.4, Y4.1, Y4.2, Y4.4; no longer U8. (VOUT)
- net ING12V+: now also J1.1 (Pin_1)
- net at C3.2, U11.8 (OSC2): now also Y1.3
- net at C4.2, U11.9 (OSC1): now also Y1.1
- net at JP2.2 (B), U7.5 (VREF): now also U6.5 (VREF)
- net CAN LISTEN L: now reaches U7.6 (CANL)
- net CAN LISTEN L: now also J1.3 (Pin_3)
- net CAN LISTEN H: now reaches U7.7 (CANH)
- net CAN LISTEN H: now also J1.4 (Pin_4)
- net OBD2 CAN L: now reaches U6.6 (CANL)
- net OBD2 CAN L: now also J1.5 (Pin_5)
- net OBD2 CAN H: now reaches U6.7 (CANH)
- net OBD2 CAN H: now also J1.6 (Pin_6)
- net at C1.2, U10.8 (OSC2): now also Y4.3
- new net: F1.2, J1.7 (Pin_7)

Commit message: pcb work
Parts:
- added D10: 1N5819HW-7-F, Diode_SMD:D_SOD-123, symbol Device:D
- added D11, D12: SD05_SOD323, Diode_SMD:D_SOD-523, symbol Diode:SD05_SOD323
- added D13: STS521050B331-EA, Diode_SMD:D_SOD-523, symbol Diode:SD05_SOD323
- added J2, J3, J4, J5, J6, J7, J8, J9: Conn_01x01, TestPoint:TestPoint_THTPad_1.0x1.0mm_Drill0.5mm, symbol Connector_Generic:Conn_01x01
- added P1: USB_C_Plug, Connector_USB:USB_C_Receptacle_GCT_USB4085, symbol Connector:USB_C_Plug
- added R14, R15: 120R, Resistor_SMD:R_0805_2012Metric, symbol Device:R
- added R16, R17: 5.1k, Resistor_SMD:R_0805_2012Metric, symbol Device:R
- C1, C2, C3, C4: footprint (none) -> Capacitor_SMD:C_0805_2012Metric
- D1, D2, D3, D4, D5, D6, D7, D8: footprint (none) -> LED_0602:LED_QBLP617-IW
- D9: footprint (none) -> Diode_SMD:D_0805_2012Metric
- F1: footprint (none) -> Fuse:Fuseholder_Littelfuse_Nano2_154x
- Q1: value NPN -> BC817; footprint (none) -> Package_TO_SOT_SMD:SOT-323_SC-70
- R1, R10, R11, R12, R13, R2, R3, R4, R5, R6, R7, R8, R9: footprint (none) -> Resistor_SMD:R_0805_2012Metric
- Y1, Y4: footprint Crystal:Crystal_SMD_3225-4Pin_3.2x2.5mm_HandSoldering -> Crystal:Crystal_SMD_3225-4Pin_3.2x2.5mm
Connections:
- net +12V: now also D10.1 (K)
- net CAN LISTEN H: now also R14.1
- net CAN LISTEN L: now also R14.2
- net GND: now also D11.1 (A1), D12.1 (A1), D13.2 (A2), P1.A1 (GND), P1.A12 (GND), P1.B1 (GND), P1.B12 (GND), P1.S1 (SHIELD), R16.1, R17.1; no longer C2.2, U10.9 (OSC1), Y4.1
- net OBD2 CAN H: now also R15.1
- net OBD2 CAN L: now also R15.2
- net at U4.15 (CS8): now also J9.1 (Pin_1)
- net at U4.16 (CS7): now also J8.1 (Pin_1)
- net at U4.17 (CS6): now also J7.1 (Pin_1)
- net at U4.18 (CS5): now also J6.1 (Pin_1)
- net at U4.19 (CS4): now also J5.1 (Pin_1)
- net at U4.20 (CS3): now also J4.1 (Pin_1)
- net at U4.21 (CS2): now also J3.1 (Pin_1)
- net at U4.22 (CS1): now also J2.1 (Pin_1)
- net at U9.17 (GPIO12/USB_D-): now also D12.2 (A2), P1.A7 (D-)
- net at U9.18 (GPIO13/USB_D+): now also D13.1 (A1), P1.A6 (D+)
- new net: C2.2, U10.9 (OSC1), Y4.1
- new net: D10.2 (A), D11.2 (A2), P1.A4 (VBUS), P1.A9 (VBUS), P1.B4 (VBUS), P1.B9 (VBUS)
- new net: P1.B5 (VCONN), R16.2
- new net: P1.A5 (CC), R17.2

Commit message: finall pcb
Parts:
- removed J1: Conn_01x07_Pin, Connector_PinHeader_2.54mm:PinHeader_1x07_P2.54mm_Horizontal, symbol Connector:Conn_01x07_Pin
- removed P1: USB_C_Plug, Connector_USB:USB_C_Receptacle_GCT_USB4085, symbol Connector:USB_C_Plug
- added C10, C11, C5, C6, C7, C8, C9: 100nF, Capacitor_SMD:C_0603_1608Metric, symbol Device:C
- added C12, C13, C14, C17: 10uF, Capacitor_SMD:C_0805_2012Metric, symbol Device:C
- added C15, C16: 100uF, Capacitor_SMD:C_1206_3216Metric, symbol Device:C
- added D14: LED, LED_0602:LED_QBLP617-IW, symbol Device:LED
- added J10: USB_C_Receptacle_USB2.0_16P, Connector_USB:USB_C_Receptacle_GCT_USB4085, symbol Connector:USB_C_Receptacle_USB2.0_16P
- added J11: MEM2085-00-115-00-A_REV0.2, MEM2085:GCT_MEM2085-00-115-00-A_REV0.2, symbol MEM2085:MEM2085-00-115-00-A_REV0.2
- added J12, J13, J14, J15, J16, J17, J18: Conn_01x01, TestPoint:TestPoint_THTPad_1.0x1.0mm_Drill0.5mm, symbol Connector_Generic:Conn_01x01
- added R18, R19: R, Resistor_SMD:R_0805_2012Metric, symbol Device:R
- J2, J3, J4, J5, J6, J7, J8, J9: footprint TestPoint:TestPoint_THTPad_1.0x1.0mm_Drill0.5mm -> TestPoint:TestPoint_Pad_1.0x1.0mm
Connections:
- net +3.3V: now also C10.1, C11.1, C12.1, C13.1, C14.1, C15.1, C16.1, C5.1, C6.1, C7.1, C8.1, C9.1, J11.P4 (VDD), R18.2, R19.1
- net CAN LISTEN H: now also J15.1 (Pin_1)
- net CAN LISTEN L: now also J16.1 (Pin_1)
- net CSCAN: now also U9.30 (U0RXD/GPIO17); no longer U9.31 (U0TXD/GPIO16)
- net CSCAN2: now also U9.31 (U0TXD/GPIO16); no longer U9.30 (U0RXD/GPIO17)
- net GND: now also C10.2, C11.2, C12.2, C13.2, C14.2, C15.2, C16.2, C17.2, C5.2, C6.2, C7.2, C8.2, C9.2, J10.A1 (GND), J10.A12 (GND), J10.B1 (GND), J10.B12 (GND), J10.S1 (SHIELD), J11.G1 (GND), J11.G10 (GND__9), J11.G2 (GND__1), J11.G3 (GND__2), J11.G4 (GND__3), J11.G5 (GND__4), J11.G6 (GND__5), J11.G7 (GND__6), J11.G8 (GND__7), J11.G9 (GND__8), J11.P6 (VSS), J17.1 (Pin_1)
- net ING12V+: now also J18.1 (Pin_1)
- net MISO: now also J11.P7 (DAT0)
- net MOSI: now also J11.P3 (CMD)
- net OBD2 CAN H: now also J14.1 (Pin_1)
- net OBD2 CAN L: now also J13.1 (Pin_1)
- net SCLK: now also J11.P5 (CLK)
- net at D10.2 (A), D11.2 (A2): now also J10.A4 (VBUS), J10.A9 (VBUS), J10.B4 (VBUS), J10.B9 (VBUS)
- net at D13.1 (A1), U9.18 (GPIO13/USB_D+): now also J10.A6 (D+), J10.B6 (D+)
- net at U9.12 (GPIO0/ADC1_CH0/XTAL_32K_P): now also D14.2 (A)
- net at D12.2 (A2), U9.17 (GPIO12/USB_D-): now also J10.A7 (D-), J10.B7 (D-)
- net CSSDCARD: now reaches U9.23 (GPIO9)
- net CSSDCARD: now also J11.CD
- net at U9.8 (EN/CHIP_PU): now also C17.1, R19.2
- net at R16.2: now also J10.B5 (CC2)
- net at F1.2: now also J12.1 (Pin_1)
- net at R17.2: now also J10.A5 (CC1)
- new net: D14.1 (K), R18.1

Commit message: deps and pcb update
Parts:
- R1: value R -> 220R
- R10, R18, R3, R4, R5, R6, R7, R8, R9: value R -> 65R
- R11, R19, R2: value R -> 10k
- R12: value R -> 4.7k
- R13: value R -> 1k
Changed lines of the file:
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@@
 			)
 		)
-		(property "Value" "R"
+		(property "Value" "10k"
 			(at 518.16 233.6799 0)
 			(effects
@@
 			)
 		)
-		(property "Value" "R"
+		(property "Value" "65R"
 			(at 580.39 297.18 90)
 			(effects
@@
 			)
 		)
-		(property "Value" "R"
+		(property "Value" "1k"
 			(at 491.49 478.79 90)
 			(effects
@@
 			)
 		)
-		(property "Value" "R"
+		(property "Value" "65R"
 			(at 580.39 281.94 90)
 			(effects
@@
 			)
 		)
-		(property "Value" "R"
+		(property "Value" "4.7k"
 			(at 491.49 466.09 90)
 			(effects
@@
 			)
 		)
-		(property "Value" "R"
+		(property "Value" "65R"
 			(at 580.39 293.37 90)
 			(effects
@@
 			)
 		)
-		(property "Value" "R"
+		(property "Value" "10k"
 			(at 358.14 237.4899 0)
 			(effects
@@
 			)
 		)
-		(property "Value" "R"
+		(property "Value" "220R"
 			(at 500.38 238.7599 0)
 			(effects
@@
 			)
 		)
-		(property "Value" "R"
+		(property "Value" "65R"
 			(at 452.12 285.75 90)
 			(effects
@@
 			)
 		)
-		(property "Value" "R"
+		(property "Value" "65R"
 			(at 580.39 289.56 90)
 			(effects
@@
 			)
 		)
-		(property "Value" "R"
+		(property "Value" "10k"
 			(at 452.12 283.21 90)
 			(effects
@@
 			)
 		)
-		(property "Value" "R"
+		(property "Value" "65R"
 			(at 580.39 278.13 90)
 			(effects
@@
 			)
 		)
-		(property "Value" "R"
+		(property "Value" "65R"
 			(at 580.39 274.32 90)
 			(effects
@@
 			)
 		)
-		(property "Value" "R"
+		(property "Value" "65R"
 			(at 580.39 285.75 90)
 			(effects
@@
 			)
 		)
-		(property "Value" "R"
+		(property "Value" "65R"
 			(at 580.39 270.51 90)
 			(effects
