File: pcb/KIA-OBD2-DISPLAY/KIA-OBD2-DISPLAY.kicad_sch (KiCad schematic)
At the start: 81 parts, among them J10 USB_C_Receptacle_USB2.0_16P, J11 MEM2085-00-115-00-A_REV0.2, J12 Conn_01x01, J13 Conn_01x01, J14 Conn_01x01, J15 Conn_01x01, J16 Conn_01x01, J17 Conn_01x01, J18 Conn_01x01, J2 Conn_01x01, J3 Conn_01x01, J4 Conn_01x01, J5 Conn_01x01, J6 Conn_01x01, J7 Conn_01x01, J8 Conn_01x01, J9 Conn_01x01, Q1 BC817, U10 MCP2515-xST, U11 MCP2515-xST, U4 CAP1188-1-CP-TR, U6 TJA1050, U7 TJA1050, U9 ESP32-C6-MINI-1/U, Y1 Crystal_GND24_Small, Y4 Crystal_GND24_Small

Commit message: more pcb work
Parts:
- U1, U2, U8: value ~ -> (none)
