File: pcb/KIA-OBD2-DISPLAY/KIA-OBD2-DISPLAY.kicad_pcb (KiCad board)
At the start: 2 copper layers, 1 part, among them U3 ESP32-C3-DevKitM-1

Commit message: run update
Parts:
- added U5: MCP2515-xSO, Package_SO:SOIC-18W_7.5x11.6mm_P1.27mm, F.Cu at (130.8, 90.5)
- added U9: ESP32-C6-MINI-1/U, PCM_Espressif:ESP32-C6-MINI-1, F.Cu at (117.0, 92.9)

Commit message: pcb 3d work
Parts:
- removed U3: ESP32-C3-DevKitM-1, PCM_Espressif:ESP32-C3-DevKitM-1
- removed U5: MCP2515-xSO, Package_SO:SOIC-18W_7.5x11.6mm_P1.27mm
- added U1: ~, SH1122:SH1122, F.Cu at (159.4, 78.0)
- added U10: MCP2515-xST, Package_SO:TSSOP-20_4.4x6.5mm_P0.65mm, B.Cu at (115.9, 84.8)
- added U11: MCP2515-xST, Package_SO:TSSOP-20_4.4x6.5mm_P0.65mm, B.Cu at (105.0, 84.8)
- added U2: ~, SH1122:SH1122, F.Cu at (159.3, 97.0)
- added U4: CAP1188-1-CP-TR, CAP1188:QFN50P400X400X90-25N, B.Cu at (208.9, 82.0)
- added U6: TJA1050, TJA1050:SOT96-1, B.Cu at (116.1, 93.6)
- added U7: TJA1050, TJA1050:SOT96-1, B.Cu at (105.5, 93.5)
- U9: moved to B.Cu
- moved U9 105.6 mm to (222.5, 87.4), turned to 90 degrees
Connections:
- net Net-(U9-GND-Pad1) renamed GND
- U9 pad 10: unconnected-(U9-MTDI/GPIO5/ADC1_CH5-Pad10) -> /INTING
- U9 pad 13: unconnected-(U9-GPIO1/ADC1_CH1/XTAL_32K_N-Pad13) -> /INTCAN2
- U9 pad 15: unconnected-(U9-MTCK/GPIO6/ADC1_CH6-Pad15) -> /SCLK
- U9 pad 16: unconnected-(U9-MTDO/GPIO7-Pad16) -> /MOSI
- U9 pad 24: unconnected-(U9-GPIO18-Pad24) -> /CSD1
- U9 pad 25: unconnected-(U9-GPIO19-Pad25) -> /CSD2
- U9 pad 26: /MISO -> /CSCAP
- U9 pad 28: unconnected-(U9-GPIO22-Pad28) -> /REST
- U9 pad 29: unconnected-(U9-GPIO23-Pad29) -> /DC
- U9 pad 3: unconnected-(U9-3V3-Pad3) -> +3.3V
- U9 pad 30: unconnected-(U9-U0RXD/GPIO17-Pad30) -> /CSCAN2
- U9 pad 31: unconnected-(U9-U0TXD/GPIO16-Pad31) -> /CSCAN
- U9 pad 5: unconnected-(U9-GPIO2/ADC1_CH2-Pad5) -> /MISO
- U9 pad 6: unconnected-(U9-GPIO3/ADC1_CH3-Pad6) -> /INTCAP
- U9 pad 9: unconnected-(U9-MTMS/GPIO4/ADC1_CH4-Pad9) -> /INTCAN
Other:
- board outline added: 132.1 x 19 mm

Commit message: pcb update
Parts:
- added J1: Conn_01x07_Pin, Connector_PinHeader_2.54mm:PinHeader_1x07_P2.54mm_Horizontal, F.Cu at (98.8, 95.1)
- added JP2: VREF 3.3V, Jumper:SolderJumper-2_P1.3mm_Open_RoundedPad1.0x1.5mm, F.Cu at (122.5, 94.9)
- added U8: ~, D24V10F3:D24V10F3, B.Cu at (142.7, 80.8)
- added Y1: Crystal_GND24_Small, Crystal:Crystal_SMD_3225-4Pin_3.2x2.5mm_HandSoldering, F.Cu at (148.9, 83.4)
- added Y4: Crystal_GND24_Small, Crystal:Crystal_SMD_3225-4Pin_3.2x2.5mm_HandSoldering, F.Cu at (148.9, 89.0)
- moved U1 19.2 mm to (159.3, 97.2), turned to 180 degrees
- moved U2 19.0 mm to (159.4, 78.0), turned to 0 degrees
Connections:
- U10 pad 9: Net-(U10-OSC1) -> GND
- U6 pad 5: Net-(JP1-B) -> Net-(JP2-B)
- U6 pad 6: unconnected-(U6-CANL-Pad6) -> /OBD2 CAN L
- U6 pad 7: unconnected-(U6-CANH-Pad7) -> /OBD2 CAN H
- U7 pad 6: unconnected-(U7-CANL-Pad6) -> /CAN LISTEN L
- U7 pad 7: unconnected-(U7-CANH-Pad7) -> /CAN LISTEN H

Commit message: pcb work
Parts:
- added C1: 22pF, Capacitor_SMD:C_0805_2012Metric, F.Cu at (165.9, 85.2)
- added C2: 22pF, Capacitor_SMD:C_0805_2012Metric, F.Cu at (165.9, 91.5)
- added C3: 22pF, Capacitor_SMD:C_0805_2012Metric, F.Cu at (177.3, 85.3)
- added C4: 22pF, Capacitor_SMD:C_0805_2012Metric, F.Cu at (177.3, 91.6)
- added D1: LED, LED_0602:LED_QBLP617-IW, B.Cu at (217.5, 78.8)
- added D10: 1N5819HW-7-F, Diode_SMD:D_SOD-123, F.Cu at (204.3, 89.4)
- added D11: SD05_SOD323, Diode_SMD:D_SOD-523, F.Cu at (209.1, 93.2)
- added D12: SD05_SOD323, Diode_SMD:D_SOD-523, F.Cu at (212.6, 91.0)
- added D13: STS521050B331-EA, Diode_SMD:D_SOD-523, F.Cu at (211.2, 92.0)
- added D2: LED, LED_0602:LED_QBLP617-IW, B.Cu at (203.9, 78.9)
- added D3: LED, LED_0602:LED_QBLP617-IW, B.Cu at (190.5, 78.9)
- added D4: LED, LED_0602:LED_QBLP617-IW, B.Cu at (173.8, 78.8)
- added D5: LED, LED_0602:LED_QBLP617-IW, B.Cu at (151.9, 79.0)
- added D6: LED, LED_0602:LED_QBLP617-IW, B.Cu at (137.7, 79.0)
- added D7: LED, LED_0602:LED_QBLP617-IW, B.Cu at (123.7, 79.0)
- added D8: LED, LED_0602:LED_QBLP617-IW, B.Cu at (110.0, 79.0)
- added D9: D, Diode_SMD:D_0805_2012Metric, F.Cu at (115.1, 82.6)
- added F1: Fuse_Small, Fuse:Fuseholder_Littelfuse_Nano2_154x, F.Cu at (129.2, 93.8)
- added J2: Conn_01x01, TestPoint:TestPoint_THTPad_1.0x1.0mm_Drill0.5mm, F.Cu at (214.6, 78.0)
- added J3: Conn_01x01, TestPoint:TestPoint_THTPad_1.0x1.0mm_Drill0.5mm, F.Cu at (201.0, 78.0)
- added J4: Conn_01x01, TestPoint:TestPoint_THTPad_1.0x1.0mm_Drill0.5mm, F.Cu at (187.5, 78.0)
- added J5: Conn_01x01, TestPoint:TestPoint_THTPad_1.0x1.0mm_Drill0.5mm, F.Cu at (170.9, 78.0)
- added J6: Conn_01x01, TestPoint:TestPoint_THTPad_1.0x1.0mm_Drill0.5mm, F.Cu at (148.8, 78.0)
- added J7: Conn_01x01, TestPoint:TestPoint_THTPad_1.0x1.0mm_Drill0.5mm, F.Cu at (134.6, 78.0)
- added J8: Conn_01x01, TestPoint:TestPoint_THTPad_1.0x1.0mm_Drill0.5mm, F.Cu at (120.7, 78.0)
- added J9: Conn_01x01, TestPoint:TestPoint_THTPad_1.0x1.0mm_Drill0.5mm, F.Cu at (106.9, 78.0)
- added P1: USB_C_Plug, Connector_USB:USB_C_Receptacle_GCT_USB4085, F.Cu at (211.1, 87.0)
- added Q1: BC817, Package_TO_SOT_SMD:SOT-323_SC-70, F.Cu at (149.0, 94.7)
- added R1: R, Resistor_SMD:R_0805_2012Metric, F.Cu at (149.0, 92.4)
- added R10: R, Resistor_SMD:R_0805_2012Metric, F.Cu at (139.3, 95.2)
- added R11: R, Resistor_SMD:R_0805_2012Metric, F.Cu at (223.6, 95.1)
- added R12: R, Resistor_SMD:R_0805_2012Metric, F.Cu at (115.1, 80.6)
- added R13: R, Resistor_SMD:R_0805_2012Metric, F.Cu at (111.7, 81.2)
- added R14: 120R, Resistor_SMD:R_0805_2012Metric, F.Cu at (187.5, 80.8)
- added R15: 120R, Resistor_SMD:R_0805_2012Metric, F.Cu at (177.3, 82.6)
- added R16: 5.1k, Resistor_SMD:R_0805_2012Metric, F.Cu at (200.9, 84.2)
- added R17: 5.1k, Resistor_SMD:R_0805_2012Metric, F.Cu at (209.4, 90.8)
- added R2: R, Resistor_SMD:R_0805_2012Metric, F.Cu at (145.5, 95.0)
- added R3: R, Resistor_SMD:R_0805_2012Metric, F.Cu at (148.6, 83.0)
- added R4: R, Resistor_SMD:R_0805_2012Metric, F.Cu at (146.6, 83.0)
- added R5: R, Resistor_SMD:R_0805_2012Metric, F.Cu at (144.6, 83.0)
- added R6: R, Resistor_SMD:R_0805_2012Metric, F.Cu at (142.7, 83.0)
- added R7: R, Resistor_SMD:R_0805_2012Metric, F.Cu at (139.3, 89.2)
- added R8: R, Resistor_SMD:R_0805_2012Metric, F.Cu at (139.3, 91.2)
- added R9: R, Resistor_SMD:R_0805_2012Metric, F.Cu at (139.3, 93.2)
- U10, U11, U4, U6, U7, U8, U9: moved to F.Cu
- Y1, Y4: footprint Crystal:Crystal_SMD_3225-4Pin_3.2x2.5mm_HandSoldering -> Crystal:Crystal_SMD_3225-4Pin_3.2x2.5mm
- moved U7 78.3 mm to (182.8, 80.7)
- moved U11 78.1 mm to (183.0, 86.8), turned to 0 degrees
- moved U4 65.0 mm to (144.3, 88.6), turned to -90 degrees
- moved U6 57.0 mm to (171.6, 80.7)
- moved JP2 56.9 mm to (177.3, 79.6)
- moved U10 55.8 mm to (171.7, 86.8), turned to 0 degrees
- moved U8 37.0 mm to (105.8, 83.9), turned to 0 degrees
- moved Y1 28.8 mm to (177.3, 88.5), turned to 90 degrees
- moved Y4 17.0 mm to (165.9, 88.3), turned to 90 degrees
- moved J1 5.33 mm to (104.1, 95.3)
- moved U9 0.61 mm to (221.9, 87.3), turned to -90 degrees
Connections:
- U10 pad 9: GND -> Net-(U10-OSC1)
- U4 pad 15: unconnected-(U4-CS8-Pad15) -> Net-(J9-Pin_1)
- U4 pad 16: unconnected-(U4-CS7-Pad16) -> Net-(J8-Pin_1)
- U4 pad 17: unconnected-(U4-CS6-Pad17) -> Net-(J7-Pin_1)
- U4 pad 18: unconnected-(U4-CS5-Pad18) -> Net-(J6-Pin_1)
- U4 pad 19: unconnected-(U4-CS4-Pad19) -> Net-(J5-Pin_1)
- U4 pad 20: unconnected-(U4-CS3-Pad20) -> Net-(J4-Pin_1)
- U4 pad 21: unconnected-(U4-CS2-Pad21) -> Net-(J3-Pin_1)
- U4 pad 22: unconnected-(U4-CS1-Pad22) -> Net-(J2-Pin_1)
- U9 pad 17: unconnected-(U9-GPIO12/USB_D--Pad17) -> Net-(D12-A2)
- U9 pad 18: unconnected-(U9-GPIO13/USB_D+-Pad18) -> Net-(D13-A1)
- Y4 pad 1: GND -> Net-(U10-OSC1)
Routing:
- net /INTING: track 0.00 -> 141.7 mm, vias 0 -> 5
- net /REST: track 0.00 -> 108.9 mm, vias 0 -> 7
- net +12V: track 0.00 -> 102.0 mm, vias 0 -> 2
- net /CAN LISTEN H: track 0.00 -> 97.2 mm, vias 0 -> 2
- net /CAN LISTEN L: track 0.00 -> 95.2 mm, vias 0 -> 2
- net /OBD2 CAN H: track 0.00 -> 83.6 mm, vias 0 -> 2
- net /OBD2 CAN L: track 0.00 -> 83.4 mm, vias 0 -> 2
- net /SCLK: track 0.00 -> 78.7 mm, vias 0 -> 2
- net /CSD1: track 0.00 -> 78.5 mm, vias 0 -> 1
- net /DC: track 0.00 -> 76.7 mm, vias 0 -> 1
- net /MOSI: track 0.00 -> 69.3 mm, vias 0 -> 3
- net /CSCAN: track 0.00 -> 58.4 mm
- net /CSD2: track 0.00 -> 56.3 mm, vias 0 -> 1
- net /MISO: track 0.00 -> 52.0 mm, vias 0 -> 2
- net Net-(J9-Pin_1): track 0.00 -> 48.8 mm, vias 0 -> 3
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- added copper zone on B.Cu, net +3.3V
- added copper zone on F.Cu, net GND
Other:
- outline, holes or cut-outs redrawn

Commit message: 4  layer pcb
Parts:
- moved R4 0.33 mm to (146.6, 82.7)
- moved R6 0.33 mm to (142.7, 82.7)
- moved R3 0.33 mm to (148.6, 82.7)
- moved R5 0.33 mm to (144.6, 82.7)
Routing:
- net /MISO: track 52.0 -> 154.3 mm, vias 2 -> 4
- net /SCLK: track 78.7 -> 98.5 mm, vias 2 -> 4
- net Net-(J6-Pin_1): track 16.5 -> 35.1 mm
- net Net-(D4-K): track 0.00 -> 15.0 mm
- net /MOSI: track 69.3 -> 82.9 mm, vias 3 -> 5
- net Net-(D3-K): track 0.00 -> 12.4 mm
- net Net-(D2-K): track 0.00 -> 9.92 mm
- net Net-(D1-K): track 0.00 -> 6.31 mm
- net Net-(U4-LED4): track 7.54 -> 5.24 mm
- net /REST: track 108.9 -> 111.0 mm
- net /CSCAP: track 0.00 -> 1.68 mm
- net /DC: track 76.7 -> 75.4 mm
- net /CSD1: track 78.5 -> 77.5 mm
- net Net-(U4-LED1): track 6.43 -> 7.15 mm
Other:
- copper layers 2 -> 4

Commit message: finall pcb
Parts:
- removed J1: Conn_01x07_Pin, Connector_PinHeader_2.54mm:PinHeader_1x07_P2.54mm_Horizontal
- removed P1: USB_C_Plug, Connector_USB:USB_C_Receptacle_GCT_USB4085
- added C10: 100nF, Capacitor_SMD:C_0603_1608Metric, F.Cu at (181.0, 91.1)
- added C11: 100nF, Capacitor_SMD:C_0603_1608Metric, F.Cu at (187.7, 85.5)
- added C12: 10uF, Capacitor_SMD:C_0805_2012Metric, F.Cu at (220.2, 95.1)
- added C13: 10uF, Capacitor_SMD:C_0805_2012Metric, F.Cu at (129.2, 94.3)
- added C14: 10uF, Capacitor_SMD:C_0805_2012Metric, F.Cu at (223.1, 79.5)
- added C15: 100uF, Capacitor_SMD:C_1206_3216Metric, F.Cu at (190.8, 94.0)
- added C16: 100uF, Capacitor_SMD:C_1206_3216Metric, F.Cu at (211.1, 95.1)
- added C17: 10uF, Capacitor_SMD:C_0805_2012Metric, F.Cu at (202.6, 93.4)
- added C5: 100nF, Capacitor_SMD:C_0603_1608Metric, F.Cu at (215.3, 94.9)
- added C6: 100nF, Capacitor_SMD:C_0603_1608Metric, F.Cu at (143.0, 95.3)
- added C7: 100nF, Capacitor_SMD:C_0603_1608Metric, F.Cu at (153.2, 92.7)
- added C8: 100nF, Capacitor_SMD:C_0603_1608Metric, F.Cu at (164.5, 82.5)
- added C9: 100nF, Capacitor_SMD:C_0603_1608Metric, F.Cu at (169.7, 91.1)
- added D14: LED, LED_0602:LED_QBLP617-IW, F.Cu at (206.2, 95.4)
- added J10: USB_C_Receptacle_USB2.0_16P, Connector_USB:USB_C_Receptacle_GCT_USB4085, F.Cu at (211.1, 87.0)
- added J11: MEM2085-00-115-00-A_REV0.2, MEM2085:GCT_MEM2085-00-115-00-A_REV0.2, F.Cu at (194.6, 88.1)
- added J12: Conn_01x01, TestPoint:TestPoint_THTPad_1.0x1.0mm_Drill0.5mm, F.Cu at (129.2, 86.2)
- added J13: Conn_01x01, TestPoint:TestPoint_THTPad_1.0x1.0mm_Drill0.5mm, B.Cu at (131.2, 84.2)
- added J14: Conn_01x01, TestPoint:TestPoint_THTPad_1.0x1.0mm_Drill0.5mm, F.Cu at (131.2, 86.2)
- added J15: Conn_01x01, TestPoint:TestPoint_THTPad_1.0x1.0mm_Drill0.5mm, F.Cu at (133.2, 84.2)
- added J16: Conn_01x01, TestPoint:TestPoint_THTPad_1.0x1.0mm_Drill0.5mm, F.Cu at (133.2, 86.2)
- added J17: Conn_01x01, TestPoint:TestPoint_THTPad_1.0x1.0mm_Drill0.5mm, B.Cu at (129.2, 84.2)
- added J18: Conn_01x01, TestPoint:TestPoint_THTPad_1.0x1.0mm_Drill0.5mm, B.Cu at (127.1, 83.1)
- added R18: R, Resistor_SMD:R_0805_2012Metric, F.Cu at (206.0, 93.5)
- added R19: R, Resistor_SMD:R_0805_2012Metric, F.Cu at (204.1, 91.5)
- J2, J3, J4, J5, J6, J7, J8, J9: footprint TestPoint:TestPoint_THTPad_1.0x1.0mm_Drill0.5mm -> TestPoint:TestPoint_Pad_1.0x1.0mm; moved to B.Cu
- moved J2 43.7 mm to (170.9, 79.0), turned to 180 degrees
- moved J5 43.7 mm to (214.6, 79.0), turned to 180 degrees
- moved J9 41.9 mm to (148.8, 79.0), turned to 180 degrees
- moved D8 26.8 mm to (134.4, 90.1), turned to 90 degrees
- moved U8 25.8 mm to (128.1, 96.8), turned to 180 degrees
- moved J6 18.3 mm to (130.6, 79.0), turned to 180 degrees
- moved R13 15.5 mm to (127.1, 80.3), turned to -90 degrees
- moved R12 14.8 mm to (129.9, 80.3)
- moved D9 14.8 mm to (129.9, 82.2)
- moved J8 14.0 mm to (134.6, 79.0), turned to 180 degrees
- moved D7 13.6 mm to (132.6, 89.2), turned to 90 degrees
- moved J4 13.5 mm to (201.0, 79.0), turned to 180 degrees
- moved J3 13.5 mm to (187.5, 79.0), turned to 180 degrees
- moved R10 12.3 mm to (139.2, 82.9), turned to -90 degrees
- moved R9 10.5 mm to (141.2, 82.9), turned to -90 degrees
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Connections:
- U9 pad 12: unconnected-(U9-GPIO0/ADC1_CH0/XTAL_32K_P-Pad12) -> Net-(D14-A)
- U9 pad 23: unconnected-(U9-GPIO9-Pad23) -> /CSSDCARD
- U9 pad 30: /CSCAN2 -> /CSCAN
- U9 pad 31: /CSCAN -> /CSCAN2
- U9 pad 8: unconnected-(U9-EN/CHIP_PU-Pad8) -> Net-(U9-EN/CHIP_PU)
Routing:
- net /INTCAP: track 0.00 -> 87.6 mm, vias 1 -> 2
- net Net-(J5-Pin_1): track 0.00 -> 87.3 mm, vias 0 -> 2
- net /CSCAP: track 1.68 -> 77.0 mm, vias 0 -> 2
- net Net-(D1-K): track 6.31 -> 78.3 mm, vias 0 -> 2
- net Net-(J4-Pin_1): track 0.00 -> 68.5 mm, vias 0 -> 2
- net Net-(J3-Pin_1): track 0.00 -> 56.7 mm, vias 0 -> 2
- net /MOSI: track 82.9 -> 138.1 mm, vias 5 -> 6
- net Net-(D2-K): track 9.92 -> 59.1 mm, vias 0 -> 2
- net /INTING: track 141.7 -> 94.8 mm, vias 5 -> 2
- net Net-(J2-Pin_1): track 0.00 -> 37.7 mm, vias 0 -> 2
- net Net-(U9-EN/CHIP_PU): track 0.00 -> 35.8 mm, vias 0 -> 2
- net /MISO: track 154.3 -> 119.5 mm, vias 4 -> 5
- net /CAN LISTEN H: track 97.2 -> 62.9 mm, vias 2 -> 3
- net Net-(J9-Pin_1): track 48.8 -> 15.8 mm, vias 3 -> 2
- net Net-(D3-K): track 12.4 -> 42.6 mm, vias 0 -> 2
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- added copper zone on In2.Cu, net +3.3V
- added copper zone on In1.Cu, net GND
Other:
- board size 132.1 x 19 mm -> 99.8 x 19.6 mm
- rule pad_to_mask_clearance: 0 -> 0.038
- rule solder_mask_min_width: 0.1016 -> 0.1

Commit message: deps and pcb update
Parts:
- R10, R18, R3, R4, R5, R6, R7, R8, R9: value R -> 65R
- R11, R19: value R -> 10k
- R12: value R -> 4.7k
- R13: value R -> 1k
Changed lines of the file:
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@@
 			(layer "F.SilkS")
 		)
-		(fp_text user "${REFERENCE}"
-			(at 9.948955 6.206265 180)
-			(unlocked yes)
-			(layer "F.Fab")
-			(effects
-				(font
-					(size 1 1)
-					(thickness 0.15)
-				)
-			)
-		)
 		(pad "1" thru_hole circle
 			(at 1.27 1.27 180)
@@
 			)
 		)
-		(property "Value" "R"
+		(property "Value" "65R"
 			(at 0 1.65 0)
 			(layer "F.Fab")
@@
 			(at 0 4.2 0)
 			(layer "F.Fab")
+			(hide yes)
 			(effects
 				(font
@@
 			)
 		)
-		(property "Value" "R"
+		(property "Value" "65R"
 			(at 0 1.65 90)
 			(layer "F.Fab")
+			(hide yes)
 			(effects
 				(font
@@
 			(at 0 2.45 -90)
 			(layer "F.Fab")
+			(hide yes)
 			(effects
 				(font
@@
 			(at 0 4.2 0)
 			(layer "F.Fab")
+			(hide yes)
 			(effects
 				(font
@@
 		)
 		(property "Value" "22pF"
-			(at 0 1.68 180)
+			(at 2.754282 0.12994 -90)
 			(layer "F.Fab")
 			(effects
@@
 			)
 		)
-		(property "Value" "R"
+		(property "Value" "65R"
 			(at 0 1.65 0)
 			(layer "F.Fab")
+			(hide yes)
 			(effects
 				(font
@@
 		)
 		(property "Value" "100nF"
-			(at 0 1.43 0)
+			(at -0.902 -1.778 0)
 			(layer "F.Fab")
 			(effects
@@
 			)
 		)
-		(property "Value" "R"
+		(property "Value" "65R"
 			(at 0 1.65 0)
 			(layer "F.Fab")
+			(hide yes)
 			(effects
 				(font
@@
 			)
 		)
-		(property "Value" "R"
+		(property "Value" "65R"
 			(at 0 1.65 90)
 			(layer "F.Fab")
@@
 		)
 		(property "Value" "TJA1050"
-			(at 6.5 0.5 90)
+			(at -4.119 -0.003 180)
 			(layer "F.Fab")
 			(effects
@@
 		)
 		(property "Value" "100nF"
-			(at 0 1.43 0)
+			(at -0.114 -1.778 0)
 			(layer "F.Fab")
 			(effects
@@
 			(at 7.95 1.95 180)
 			(layer "F.Fab")
+			(hide yes)
 			(effects
 				(font
@@
 		)
 		(property "Value" "5.1k"
-			(at 0 1.65 90)
+			(at -1.858128 1.804804 90)
 			(layer "F.Fab")
 			(effects
@@
 			(at 0 1.85 0)
 			(layer "F.Fab")
-			(hide yes)
 			(effects
 				(font
@@
 			)
 		)
-		(property "Value" "R"
+		(property "Value" "10k"
 			(at 0 1.65 0)
 			(layer "F.Fab")
@@
 		)
 		(property "Value" "SD05_SOD323"
-			(at 0 1.4 0)
+			(at -3.995 5.86 0)
 			(layer "F.Fab")
-			(hide yes)
 			(effects
 				(font
@@
 		)
 		(fp_text user "${REFERENCE}"
-			(at 0 -1.3 0)
+			(at -1.963 -1.633 0)
 			(layer "F.Fab")
 			(effects
@@
 		)
 		(property "Value" "100nF"
-			(at 0 1.43 90)
+			(at 3.823 0 90)
 			(layer "F.Fab")
 			(effects
@@
 		)
 		(property "Value" "100nF"
-			(at 0 1.43 0)
+			(at -1.257 -1.778 0)
 			(layer "F.Fab")
 			(effects
@@
 			)
 		)
-		(property "Value" "R"
-			(at 0 1.65 0)
+		(property "Value" "65R"
+			(at 0 3.81 0)
 			(layer "F.Fab")
 			(effects
@@
 			)
 		)
-		(property "Value" "R"
+		(property "Value" "65R"
 			(at 0 1.65 0)
 			(layer "F.Fab")
+			(hide yes)
 			(effects
 				(font
@@
 		)
 		(property "Value" "10uF"
-			(at 0 1.68 0)
+			(at 1.649364 -2.224239 0)
 			(layer "F.Fab")
 			(effects
@@
 		)
 		(property "Value" "100nF"
-			(at 0 1.43 0)
+			(at -0.876 -1.778 0)
 			(layer "F.Fab")
 			(effects
@@
 		)
 		(property "Value" "22pF"
-			(at 0 1.68 180)
+			(at -0.018646 -1.678598 0)
 			(layer "F.Fab")
 			(effects
@@
 		)
 		(property "Value" "TJA1050"
-			(at 6.5 0.5 90)
+			(at -4.069 0.020975 180)
 			(layer "F.Fab")
 			(effects
@@
 		)
 		(property "Value" "100uF"
-			(at 0 1.85 0)
+			(at 0 -2.032 0)
 			(layer "F.Fab")
 			(effects
@@
 		)
 		(fp_text user "${REFERENCE}"
-			(at 0 -1.3 -90)
+			(at 0.068 2.665 0)
 			(layer "F.Fab")
 			(effects
@@
 		)
 		(property "Value" "5.1k"
-			(at 0 1.65 -90)
+			(at 1.646 -1.755 -90)
 			(layer "F.Fab")
-			(hide yes)
 			(effects
 				(font
@@
 		)
 		(property "Value" "10uF"
-			(at 0 1.68 0)
+			(at -0.315 -2.159 0)
 			(layer "F.Fab")
 			(effects
@@
 		)
 		(fp_text user "${REFERENCE}"
-			(at 0 -1.3 90)
+			(at -2.769 0.076 -90)
 			(layer "F.Fab")
 			(effects
@@
 		)
 		(property "Value" "10uF"
-			(at 0 1.68 0)
+			(at 0 -1.905 0)
 			(layer "F.Fab")
 			(effects
@@
 		)
 		(property "Value" "BC817"
-			(at -0.05 2.05 180)
+			(at -0.227313 -2.57776 180)
 			(layer "F.Fab")
 			(effects
@@
 			)
 		)
-		(property "Value" "R"
+		(property "Value" "4.7k"
 			(at 0 1.65 180)
 			(layer "F.Fab")
@@
 			)
 		)
-		(property "Value" "R"
+		(property "Value" "1k"
 			(at 0 1.65 90)
 			(layer "F.Fab")
@@
 		)
 		(property "Value" "120R"
-			(at 0 1.65 90)
+			(at 0.224859 -1.972484 90)
 			(layer "F.Fab")
 			(effects
@@
 			(at 12.85 -5.315 0)
 			(layer "F.Fab")
+			(hide yes)
 			(effects
 				(font
@@
 			)
 		)
-		(property "Value" "R"
+		(property "Value" "65R"
 			(at 0 1.65 90)
 			(layer "F.Fab")
+			(hide yes)
 			(effects
 				(font
@@
 			(at 0 2.45 -90)
 			(layer "F.Fab")
+			(hide yes)
 			(effects
 				(font
@@
 			(at 0 1.9 0)
 			(layer "F.Fab")
+			(hide yes)
 			(effects
 				(font
@@
 		)
 		(property "Value" "100nF"
-			(at 0 1.43 90)
+			(at 2.68 -0.508 180)
 			(layer "F.Fab")
 			(effects
@@
 		)
 		(property "Value" "100nF"
-			(at 0 1.43 90)
+			(at 3.1242 0.635 180)
 			(layer "F.Fab")
 			(effects
@@
 			)
 		)
-		(property "Value" "R"
-			(at 0 1.65 0)
+		(property "Value" "10k"
+			(at 3.106765 0.082492 0)
 			(layer "F.Fab")
 			(effects
@@
 			)
 		)
-		(property "Value" "R"
+		(property "Value" "65R"
 			(at 0 1.65 90)
 			(layer "F.Fab")
@@
 		)
 		(property "Value" "120R"
-			(at 0 1.65 90)
+			(at -5.749411 -0.122566 0)
 			(layer "F.Fab")
 			(effects
@@
 			(at 0 -1.55 0)
 			(layer "B.Fab")
+			(hide yes)
 			(effects
 				(font
@@
 			(at 0 -1.55 0)
 			(layer "B.Fab")
+			(hide yes)
 			(effects
 				(font
@@
 			(at 0 -1.55 0)
 			(layer "B.Fab")
+			(hide yes)
 			(effects
 				(font
@@
 			(at 0 -1.55 0)
 			(layer "B.Fab")
+			(hide yes)
 			(effects
 				(font
@@
 	)
 	(segment
-		(start 140.0698 87.565)
-		(end 140.0048 87.63)
+		(start 139.9906 87.565)
+		(end 139.9032 87.4776)
 		(width 0.25)
 		(layer "F.Cu")
@@
 	(segment
 		(start 140.8715 87.565)
-		(end 140.0698 87.565)
+		(end 139.9906 87.565)
 		(width 0.25)
 		(layer "F.Cu")
