File: pcb/FLEX-MIPI/FLEX-MIPI.kicad_sch (KiCad schematic)
At the start: 2 parts, among them CN1 OK-23GF030-04, J1 Conn_01x22

Commit message: avoid drawing touch at full fps
Parts:
- added C1: 10uF, Package_SO:SOIC-8_3.9x4.9mm_P1.27mm, symbol Device:C
- added C2, C3: 0.1uF, symbol Device:C
- added R1, R2, R3, R4: R, symbol Device:R
Connections:
- net +3V3: now also C1.1, C2.1, R1.1, R2.1, R3.1, R4.2
- net GND: now also C1.2, C2.2, C3.2
- net LCM_ID: now also CN1.14
- net TP_TWI2_SCK: now also R1.2
- net TP_TWI2_SDA: now also R2.2
- net VCI_EN: now also R3.2; no longer J1.5 (Pin_5)
- net CTP_INT renamed TP_INT
- net TP_INT: now also J1.5 (Pin_5)
- net CTP_RST renamed LCD_RST
- net LCD_RST: now also C3.1, R4.1

Commit message: flex mipi work
Parts:
- added TP1: TestPoint, TestPoint_SMD_1.0x0.6mm_Flex:TestPoint_SMD_1.0x0.6mm_Flex, symbol Connector:TestPoint
- C1: footprint Package_SO:SOIC-8_3.9x4.9mm_P1.27mm -> Capacitor_SMD:C_0805_2012Metric_Pad1.18x1.45mm_HandSolder
- C2, C3: footprint (none) -> Capacitor_SMD:C_0201_0603Metric_Pad0.64x0.40mm_HandSolder
- R1, R2, R3, R4: footprint (none) -> Resistor_SMD:R_0201_0603Metric_Pad0.64x0.40mm_HandSolder
Connections:
- net TP_INT: now also TP1.1
- net LCD_RST renamed RST
Changed lines of the file:
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@@
 	(wire
 		(pts
-			(xy 140.97 77.47) (xy 143.51 77.47)
+			(xy 158.75 146.05) (xy 158.75 148.59)
 		)
 		(stroke
@@
 	(wire
 		(pts
-			(xy 119.38 147.32) (xy 116.84 147.32)
+			(xy 140.97 77.47) (xy 143.51 77.47)
 		)
 		(stroke
@@
 	(wire
 		(pts
-			(xy 123.19 85.09) (xy 124.46 85.09)
+			(xy 119.38 147.32) (xy 116.84 147.32)
 		)
 		(stroke
@@
 	(wire
 		(pts
-			(xy 124.46 72.39) (xy 125.73 72.39)
+			(xy 123.19 85.09) (xy 124.46 85.09)
 		)
 		(stroke
@@
 	(wire
 		(pts
-			(xy 158.75 146.05) (xy 170.18 146.05)
+			(xy 124.46 72.39) (xy 125.73 72.39)
 		)
 		(stroke
@@
 	(wire
 		(pts
-			(xy 74.93 81.28) (xy 86.36 81.28)
-		)
-		(stroke
-			(width 0)
-			(type default)
-		)
-	)
-	(wire
-		(pts
 			(xy 123.19 74.93) (xy 125.73 74.93)
 		)
@@
 	(wire
 		(pts
-			(xy 158.75 146.05) (xy 158.75 148.59)
+			(xy 127 143.51) (xy 129.54 143.51)
 		)
 		(stroke
@@
 	(wire
 		(pts
-			(xy 127 143.51) (xy 129.54 143.51)
+			(xy 74.93 78.74) (xy 78.74 78.74)
 		)
 		(stroke
@@
 	(wire
 		(pts
-			(xy 74.93 78.74) (xy 78.74 78.74)
+			(xy 158.75 146.05) (xy 162.56 146.05)
 		)
 		(stroke
@@
 		)
 	)
+	(wire
+		(pts
+			(xy 74.93 81.28) (xy 78.74 81.28)
+		)
+		(stroke
+			(width 0)
+			(type default)
+		)
+	)
+	(wire
+		(pts
+			(xy 182.88 76.2) (xy 186.69 76.2)
+		)
+		(stroke
+			(width 0)
+			(type default)
+		)
+	)
 	(label "LCM_ID"
 		(at 123.19 102.87 180)
@@
 		)
 	)
-	(label "TP_RST"
-		(at 86.36 81.28 0)
-		(effects
-			(font
-				(size 1 1)
-				(color 221 133 0 1)
-			)
-			(justify left bottom)
-		)
-	)
 	(label "LCM_CLKN"
 		(at 123.19 74.93 180)
@@
 		)
 	)
-	(label "LCD_RST"
+	(label "RST"
 		(at 162.56 146.05 0)
 		(effects
@@
 		)
 	)
+	(label "TP_INT"
+		(at 182.88 76.2 180)
+		(effects
+			(font
+				(size 1 1)
+				(color 221 133 0 1)
+			)
+			(justify right bottom)
+		)
+	)
 	(label "LCM_D0N"
 		(at 78.74 119.38 0)
@@
 		)
 	)
-	(label "LCD_RST"
+	(label "RST"
 		(at 78.74 81.28 0)
 		(effects
@@
 		)
 	)
-	(label "LCD_RST"
+	(label "RST"
 		(at 123.19 97.79 180)
 		(effects
@@
 		)
 	)
-	(label "TP_RST"
+	(label "RST"
 		(at 144.78 90.17 0)
 		(effects
 			(font
 				(size 1 1)
-				(color 221 133 0 1)
-			)
-			(justify left bottom)
-		)
-	)
-	(label "TP_RST"
-		(at 170.18 146.05 0)
-		(effects
-			(font
-				(size 1 1)
-				(color 221 133 0 1)
+				(color 0 0 0 1)
 			)
 			(justify left bottom)
@@
 			)
 		)
-		(property "Footprint" ""
+		(property "Footprint" "Capacitor_SMD:C_0201_0603Metric_Pad0.64x0.40mm_HandSolder"
 			(at 159.7152 156.21 0)
 			(hide yes)
@@
 			)
 		)
-		(property "Footprint" ""
+		(property "Footprint" "Resistor_SMD:R_0201_0603Metric_Pad0.64x0.40mm_HandSolder"
 			(at 160.528 140.97 90)
 			(hide yes)
@@
 			)
 		)
-		(property "Footprint" ""
+		(property "Footprint" "Capacitor_SMD:C_0201_0603Metric_Pad0.64x0.40mm_HandSolder"
 			(at 91.1352 148.59 0)
 			(hide yes)
@@
 			)
 		)
-		(property "Footprint" "Package_SO:SOIC-8_3.9x4.9mm_P1.27mm"
+		(property "Footprint" "Capacitor_SMD:C_0805_2012Metric_Pad1.18x1.45mm_HandSolder"
 			(at 84.7852 148.59 0)
 			(hide yes)
@@
 	)
 	(symbol
+		(lib_id "Connector:TestPoint")
+		(at 186.69 76.2 270)
+		(unit 1)
+		(body_style 1)
+		(exclude_from_sim no)
+		(in_bom yes)
+		(on_board yes)
+		(in_pos_files yes)
+		(dnp no)
+		(fields_autoplaced yes)
+		(property "Reference" "TP1"
+			(at 191.77 74.9299 90)
+			(show_name no)
+			(do_not_autoplace no)
+			(effects
+				(font
+					(size 1.27 1.27)
+				)
+				(justify left)
+			)
+		)
+		(property "Value" "TestPoint"
+			(at 191.77 77.4699 90)
+			(show_name no)
+			(do_not_autoplace no)
+			(effects
+				(font
+					(size 1.27 1.27)
+				)
+				(justify left)
+			)
+		)
+		(property "Footprint" "TestPoint_SMD_1.0x0.6mm_Flex:TestPoint_SMD_1.0x0.6mm_Flex"
+			(at 186.69 81.28 0)
+			(hide yes)
+			(show_name no)
+			(do_not_autoplace no)
+			(effects
+				(font
+					(size 1.27 1.27)
+				)
+			)
+		)
+		(property "Datasheet" ""
+			(at 186.69 81.28 0)
+			(hide yes)
+			(show_name no)
+			(do_not_autoplace no)
+			(effects
+				(font
+					(size 1.27 1.27)
+				)
+			)
+		)
+		(property "Description" "test point"
+			(at 186.69 76.2 0)
+			(hide yes)
+			(show_name no)
+			(do_not_autoplace no)
+			(effects
+				(font
+					(size 1.27 1.27)
+				)
+			)
+		)
+		(pin "1"
+		)
+		(instances
+			(project "FLEX-MIPI"
+				(path "/38ce2e03-1eb8-418d-a7f8-6a4b8bfe2962"
+					(reference "TP1")
+					(unit 1)
+				)
+			)
+		)
+	)
+	(symbol
 		(lib_id "power:+3V3")
 		(at 83.82 135.89 0)
@@
 			)
 		)
-		(property "Footprint" ""
+		(property "Footprint" "Resistor_SMD:R_0201_0603Metric_Pad0.64x0.40mm_HandSolder"
 			(at 123.19 145.288 90)
 			(hide yes)
@@
 			)
 		)
-		(property "Footprint" ""
+		(property "Footprint" "Resistor_SMD:R_0201_0603Metric_Pad0.64x0.40mm_HandSolder"
 			(at 123.19 141.478 90)
 			(hide yes)
@@
 			)
 		)
-		(property "Footprint" ""
+		(property "Footprint" "Resistor_SMD:R_0201_0603Metric_Pad0.64x0.40mm_HandSolder"
 			(at 123.19 149.098 90)
 			(hide yes)
