File: pcb/LUCKFOX-LYRA-ZEROW/LUCKFOX-LYRA-ZEROW.kicad_sch (KiCad schematic)
At the start: 3 parts, among them U1 Luckfox_Lyra_Zero_W, U2 ME54BS12-nRF54L15, U3 ME54BS01-nRF54L15

Commit message: slint upgrade
Parts:
- added U4: MCP2518FD-xQBB, Package_DFN_QFN:DFN-14-1EP_3x4.5mm_P0.65mm_EP1.65x4.25mm, symbol Interface_CAN_LIN:MCP2518FD-xQBB
Connections:
- new net: U4.15 (VSS), U4.7 (VSS)
Changed lines of the file:
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@@
+	)
+	(symbol
+		(lib_id "Interface_CAN_LIN:MCP2518FD-xQBB")
+		(at 229.87 63.5 0)
+		(unit 1)
+		(body_style 1)
+		(exclude_from_sim no)
+		(in_bom yes)
+		(on_board yes)
+		(in_pos_files yes)
+		(dnp no)
+		(fields_autoplaced yes)
+		(property "Reference" "U4"
+			(at 232.0133 48.26 0)
+			(show_name no)
+			(do_not_autoplace no)
+			(effects
+				(font
+					(size 1.27 1.27)
+				)
+				(justify left)
+			)
+		)
+		(property "Value" "MCP2518FD-xQBB"
+			(at 232.0133 50.8 0)
+			(show_name no)
+			(do_not_autoplace no)
+			(effects
+				(font
+					(size 1.27 1.27)
+				)
+				(justify left)
+			)
+		)
+		(property "Footprint" "Package_DFN_QFN:DFN-14-1EP_3x4.5mm_P0.65mm_EP1.65x4.25mm"
+			(at 231.14 77.47 0)
+			(hide yes)
+			(show_name no)
+			(do_not_autoplace no)
+			(effects
+				(font
+					(size 1.27 1.27)
+				)
+				(justify left)
+			)
+		)
+		(property "Datasheet" "https://ww1.microchip.com/downloads/aemDocuments/documents/OTH/ProductDocuments/DataSheets/External-CAN-FD-Controller-with-SPI-Interface-DS20006027B.pdf"
+			(at 231.14 80.01 0)
+			(hide yes)
+			(show_name no)
+			(do_not_autoplace no)
+			(effects
+				(font
+					(size 1.27 1.27)
+				)
+				(justify left)
+			)
+		)
+		(property "Description" "CAN FD Controller with SPI Interface, up to 8 Mbps, Vdd 2.7..5.5V,  functional safety ready, VDFN-14"
+			(at 229.87 63.5 0)
+			(hide yes)
+			(show_name no)
+			(do_not_autoplace no)
+			(effects
+				(font
+					(size 1.27 1.27)
+				)
+			)
+		)
+		(pin "8"
+		)
+		(pin "7"
+		)
+		(pin "6"
+		)
+		(pin "5"
+		)
+		(pin "4"
+		)
+		(pin "3"
+		)
+		(pin "2"
+		)
+		(pin "1"
+		)
+		(pin "15"
+		)
+		(pin "14"
+		)
+		(pin "13"
+		)
+		(pin "12"
+		)
+		(pin "11"
+		)
+		(pin "10"
+		)
+		(pin "9"
+		)
+		(instances
+			(project "LUCKFOX-LYRA-ZEROW"
+				(path "/01a1a023-e48c-458b-aa28-b9cd6c31a0a1"
+					(reference "U4")
+					(unit 1)
+				)
+			)
+		)
 	)
 	(symbol

Commit message: more pcb work
Parts:
- removed U2: ME54BS12-nRF54L15, MinewSemi_nRF54:ME54BS12_nRF54L15, symbol MinewSemi_nRF54:ME54BS12_nRF54L15
- removed U3: ME54BS01-nRF54L15, MinewSemi_nRF54:ME54BS01_nRF54L15, symbol MinewSemi_nRF54:ME54BS01_nRF54L15
- added C10, C15, C4: 10uF/50V-X5R(X7R)_1206, ETH3:C_1206(3216), symbol ETH3:C_small_PG
- added C11, C3, C9: 100nF/50V-X7R_0805, ETH3:C_0805(2012), symbol ETH3:C_small_PG
- added C12, C13, C14: 10uF/16V(25V,35V,50V)-X5R(X7R)_1206, ETH3:C_1206(3216), symbol ETH3:C_small_PG
- added C16: 10uF/50V-X5R(X7R)_1206, symbol ETH3:C_small_PG
- added CE1: 100uF/50V EEUFR1H101, EEUFR1V101(100uF/35V), EEUF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, ETH3:CE_Radial_D8.0mm_P3.50mm, symbol ETH3:C_polarized_small
- added D5: PMEG4020ER, ETH3:SOD-123F_SOD123W_CFP3, symbol ETH3:D_Schott_small_PG
- added D6: PMEG4020ER, symbol ETH3:D_Schott_small_PG
- added DL1: MPZ2012S221ATxxx (MPZ2012S331ATxxx), (BLM21PG221S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, ETH3:R_0805(2012), symbol ETH3:L_small
- added DL2: SRP7028CC-220M (SRP7028A-220M), (SRP7028AA-220M),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, ETH3:L_BOURNS_SRP7028, symbol ETH3:L_small
- added DL3: SRP7028CC-220M (SRP7028A-220M), (SRP7028AA-220M),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, symbol ETH3:L_small
- added DT1: P6SMB33A, ETH3:D_SMB, symbol ETH3:D_Zen_PESD_small
- added F1: Fuse_Small, Fuse:Fuseholder_Littelfuse_Nano2_154x, symbol Device:Fuse_Small
- added J12, J13, J14, J15, J16, J17, J18: Conn_01x01, TestPoint:TestPoint_THTPad_1.0x1.0mm_Drill0.5mm, symbol Connector_Generic:Conn_01x01
- added R10, R7: (150k/1%_0805), ETH3:R_0805(2012), symbol ETH3:R_small_PG
- added R11, R12, R9: 22k/1%_0805, ETH3:R_0805(2012), symbol ETH3:R_small_PG
- added R8: 100k/1%_0805, ETH3:R_0805(2012), symbol ETH3:R_small_PG
- added RD1: 0,39R MMA02040C 3907J(G,F) (0,33R MMA02040C 3307J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, ETH3:R_MiniMELF-0204, symbol ETH3:R_small_PG
- added S1: LMR54406FDBVR (LMR54410FDBVR), (LMR54406DBVR), (L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, ETH3:SOT-23-6, symbol ETH3:LMR54406FDBVR
- added U10: RAA211403, RAA211403:SOT-23-5_L3.0-W1.7-P0.95-LS2.8-BL, symbol RAA211403:RAA2114034GP3#JA0
- added U11, U9: 74AUP2G34GW,125, Package_TO_SOT_SMD:SOT-363_SC-70-6_Handsoldering, symbol 74AUP2G34:74AUP2G34GW,125
- added U12: 74LVC2G66, RAA211403:SOT-23-5_L3.0-W1.7-P0.95-LS2.8-BL, symbol 74xGxx:74LVC2G66
- added U2: CORE52840, Core52840:BULETM-SMD_HOLYIOT-18010-NRF52840, symbol Core52840:CORE52840
- added U3, U5, U6, U8: MAX3051, Package_SO:SOIC-8_3.9x4.9mm_P1.27mm, symbol Interface_UART:MAX3051
- added U7: MCP2518FD-xQBB, Package_DFN_QFN:DFN-14-1EP_3x4.5mm_P0.65mm_EP1.65x4.25mm, symbol Interface_CAN_LIN:MCP2518FD-xQBB
Connections:
- net +3.3VA: now reaches U1.1 (3V3)
- net +3.3VA: now also U1.17 (3V3), R11.1, U12.3, U12.7, U3.3 (VDD), U5.3 (VDD), U9.5 (VCC)
- net TOUCH_INT: now reaches U1.11 (RMIO3_/_GPIO0_A3)
- net TOUCH_RST: now reaches U1.13 (RMIO4_/_GPIO0_A4)
- net GND: now reaches U1.14 (GND)
- net GND: now also U1.20 (GND), U1.25 (GND), U1.30 (GND), U1.34 (GND), U1.39 (GND), U1.6 (GND), U1.9 (GND), U4.15 (VSS), U4.7 (VSS), C10.2, C12.2, C13.2, C14.2, C15.2, C16.2, C3.2, C4.2, C9.2, CE1.2, D5.2 (A), D6.2 (A), DT1.2, J17.1 (Pin_1), R7.2, R9.2, S1.2 (GND), U10.2 (GND), U11.2 (GND), U2.1 (GND), U2.25 (GND), U2.37 (GND), U3.2 (GND), U3.8 (RS), U5.2 (GND), U5.8 (RS), U6.2 (GND), U6.8 (RS), U7.15 (VSS), U7.7 (VSS), U8.2 (GND), U8.8 (RS), U9.2 (GND)
- net LYRA_SPI1_MOSI: now reaches U1.18 (RMIO9_/_GPIO0_B1)
- net LYRA_SPI1_MOSI: now also R12.1
- net +5V: now reaches U1.2 (5V)
- net +5V: now also U1.4 (5V), C12.1, C13.1, C14.1, DL2.2, R8.1
- net LYRA_SPI1_CS1: now reaches U1.21 (RMIO7_/_GPIO0_A7)
- net LYRA_SPI1_MISO: now reaches U1.22 (RMIO10_/_GPIO0_B2)
- net LYRA_SPI1_MISO: now also R12.2, U12.1
- net LYRA_SPI1_SCLK: now reaches U1.23 (RMIO8_/_GPIO0_B0)
- net LYRA_SPI1_SCLK: now also U12.5
- net LCD_RST: now reaches U1.28 (RMIO13_/_GPIO0_B5)
- net CAN1_TX: now reaches U1.29 (RMIO25_/_GPIO1_B2)
- net CAN1_TX: now also U5.1 (TXD)
- net TOUCH_SDA: now reaches U1.3 (RMIO0_/_GPIO0_A0)
- net CAN1_RX: now reaches U1.31 (RMIO26_/_GPIO1_B3)
- net CAN1_RX: now also U5.4 (RXD)
- net LYRA_UART1_RX: now reaches U1.32 (RMIO14_/_GPIO0_B6)
- net LYRA_UART1_RX: now also U9.6 (1Y)
- net CAN0_TX: now reaches U1.33 (RMIO27_/_GPIO1_C2)
- net CAN0_TX: now also U3.1 (TXD)
- net UART0_RX: now reaches U1.36 (RMIO23_/_GPIO0_C7)
- net CAN0_RX: now reaches U1.37 (RMIO28_/_GPIO1_C3)
- net CAN0_RX: now also U3.4 (RXD)
- net UART0_TX: now reaches U1.38 (RMIO22_/_GPIO0_C6)
- net TOUCH_SCL: now reaches U1.5 (RMIO1_/_GPIO0_A1)
- net LYRA_UART1_TX: now reaches U1.7 (RMIO2_/_GPIO0_A2)
- net LYRA_UART1_TX: now also U9.3 (2A)
- net at U4.1 (TXCAN): now also U6.1 (TXD)
- net +3V3: now reaches U4.14 (VDD)
- net +3V3: now also C16.1, DL3.2, U10.1 (VOUT), U12.8 (VCC), U2.14 (VDD-nRF), U6.3 (VDD), U7.14 (VDD), U8.3 (VDD)
- net at U4.2 (RXCAN): now also U6.4 (RXD)
- new net: C10.1, C15.1, C9.1, DL1.2, R10.2, RD1.1, S1.5 (Vin), U10.4 (VIN)
- new net: C11.2, D5.1 (K), DL2.1, S1.6 (SW)
- new net: F1.2, J12.1 (Pin_1)
- new net: D6.1 (K), DL3.1, U10.5 (SW)
- new net: R10.1, U10.3 (EN)
- new net: R7.1, R8.2, R9.1, S1.3 (FB)
- new net: C11.1, S1.1 (CB)
- new net: CE1.1, RD1.2
- new net: R11.2, U12.4 (GND)
- new net: U7.1 (TXCAN), U8.1 (TXD)
- new net: U7.2 (RXCAN), U8.4 (RXD)
- new net +12V: C3.1, C4.1, DL1.1, DT1.1, F1.1
- new net 5V_EN: S1.4 (EN)
- new net CAN LISTEN H: J15.1 (Pin_1)
- new net CAN LISTEN L: J16.1 (Pin_1)
- new net ING12V+: J18.1 (Pin_1)
- new net NRF_SWDCLK: U12.6, U2.31 (SWDCLK)
- new net NRF_SWDIO: U12.2, U2.32 (SWDIO)
- new net NRF_UART_RX: U2.35 (P0.09), U9.4 (2Y)
- new net NRF_UART_TX: U2.36 (P0.10), U9.1 (1A)
- new net OBD2 CAN H: J14.1 (Pin_1)
- new net OBD2 CAN L: J13.1 (Pin_1)
- no-connect marks 0 -> 1
Other:
- moved on the sheet: U1, U4

Commit message: PCB LYRA work
Parts:
- removed CE1: 100uF/50V EEUFR1H101, EEUFR1V101(100uF/35V), EEUF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, ETH3:CE_Radial_D8.0mm_P3.50mm, symbol ETH3:C_polarized_small
- removed J12, J13, J14, J15, J16, J17, J18: Conn_01x01, TestPoint:TestPoint_THTPad_1.0x1.0mm_Drill0.5mm, symbol Connector_Generic:Conn_01x01
- removed U11: 74AUP2G34GW,125, Package_TO_SOT_SMD:SOT-363_SC-70-6_Handsoldering, symbol 74AUP2G34:74AUP2G34GW,125
- added C1, C2, C5, C6: 22pF, Capacitor_SMD:C_0805_2012Metric, symbol Device:C_Small
- added C17, C18, C20, C22, C24, C26, C28, C30, C32: 100nF/50V-X7R_0805, Capacitor_SMD:C_0805_2012Metric_Pad1.18x1.45mm_HandSolder, symbol ETH3:C_small_PG
- added C19, C21, C23, C25, C27, C29, C31, C33: 10uF/50V-X5R(X7R)_1206, Capacitor_SMD:C_1206_3216Metric_Pad1.33x1.80mm_HandSolder, symbol ETH3:C_small_PG
- added C34: 22uF / 50V, Capacitor_SMD:C_2220_5750Metric_Pad1.97x5.40mm_HandSolder, symbol ETH3:C_small_PG
- added D9: D, Diode_SMD:D_0805_2012Metric, symbol Device:D
- added J1, J3: Conn_01x07, Connector_JST:JST_GH_SM07B-GHS-TB_1x07-1MP_P1.25mm_Horizontal, symbol Connector_Generic:Conn_01x07
- added J2, J4, J5: Conn_01x05, Connector_JST:JST_GH_SM05B-GHS-TB_1x05-1MP_P1.25mm_Horizontal, symbol Connector_Generic:Conn_01x05
- added R13: 47k, Resistor_SMD:R_0805_2012Metric_Pad1.20x1.40mm_HandSolder, symbol Device:R
- added R14: 10k, Resistor_SMD:R_0805_2012Metric_Pad1.20x1.40mm_HandSolder, symbol Device:R
- added R15, R21: (no value), Resistor_SMD:R_0805_2012Metric_Pad1.20x1.40mm_HandSolder, symbol ETH3:R_small_PG
- added R16, R17, R18, R19, R20: (150k/1%_0805), Resistor_SMD:R_0805_2012Metric_Pad1.20x1.40mm_HandSolder, symbol ETH3:R_small_PG
- added U11: SN74LVC1G74DCUT, Package_SO:VSSOP-8_2.3x2mm_P0.5mm, symbol SN74LVC1G74:SN74LVC1G74DCTR
- added U13: TPS3839G33DBZT, Package_TO_SOT_SMD:SOT-23, symbol Power_Supervisor:TPS3839DBZ
- added U14: 74AUP2G34GW,125, Package_TO_SOT_SMD:SOT-363_SC-70-6_Handsoldering, symbol 74AUP2G34:74AUP2G34GW,125
- added Y4, Y5: Crystal_GND24_Small, Crystal:Crystal_SMD_3225-4Pin_3.2x2.5mm, symbol Device:Crystal_GND24_Small
- C10, C12, C13, C14, C15, C4: footprint ETH3:C_1206(3216) -> Capacitor_SMD:C_1206_3216Metric_Pad1.33x1.80mm_HandSolder
- C11, C3, C9: footprint ETH3:C_0805(2012) -> Capacitor_SMD:C_0805_2012Metric_Pad1.18x1.45mm_HandSolder
- C16: footprint (none) -> Capacitor_SMD:C_1206_3216Metric_Pad1.33x1.80mm_HandSolder
- D5: footprint ETH3:SOD-123F_SOD123W_CFP3 -> Diode_SMD:D_SOD-123F
- D6: value PMEG4020ER -> SKL16-AQ; footprint (none) -> Diode_SMD:D_SMA_Handsoldering; Wartość wyśw. MBR1060HEWS -> SKL16-AQ
- DL1: footprint ETH3:R_0805(2012) -> Inductor_SMD:L_0805_2012Metric_Pad1.05x1.20mm_HandSolder
- DL2: value SRP7028CC-220M (SRP7028A-220M), (SRP7028AA-220M), (SRP6540-220M) -> SRP7028CC-220M/150M; footprint ETH3:L_BOURNS_SRP7028 -> Inductor_SMD:L_Bourns_SRP7028A_7.3x6.6mm; Wartość wyśw. SRP7028CC-220M -> SRP7028CC-220M/150M
- DL3: value SRP7028CC-220M (SRP7028A-220M), (SRP7028AA-220M), (SRP6540-220M) -> 15uH; footprint (none) -> Inductor_SMD:L_Wuerth_MAPI-3015
- DT1: footprint ETH3:D_SMB -> Diode_SMD:D_SMB_Handsoldering
- R10, R11, R7, R8, R9: footprint ETH3:R_0805(2012) -> Resistor_SMD:R_0805_2012Metric_Pad1.20x1.40mm_HandSolder
- R12: value 22k/1%_0805 -> 1k; footprint ETH3:R_0805(2012) -> Resistor_SMD:R_0805_2012Metric_Pad1.20x1.40mm_HandSolder
- RD1: footprint ETH3:R_MiniMELF-0204 -> Resistor_SMD:R_MiniMELF_MMA-0204
- S1: footprint ETH3:SOT-23-6 -> Package_TO_SOT_SMD:SOT-23-6_Handsoldering
- U12: footprint RAA211403:SOT-23-5_L3.0-W1.7-P0.95-LS2.8-BL -> Package_SO:TSSOP-8_3x3mm_P0.65mm
- U4, U7: footprint Package_DFN_QFN:DFN-14-1EP_3x4.5mm_P0.65mm_EP1.65x4.25mm -> Package_SO:SOIC-14_3.9x8.7mm_P1.27mm
Connections:
- net +3.3VA: now also C28.1, C29.1, C30.1, C31.1, J5.4 (Pin_4), U14.5 (VCC)
- net +3V3: now also C18.1, C19.1, C20.1, C21.1, C22.1, C23.1, C24.1, C25.1, C26.1, C27.1, J2.4 (Pin_4), J3.6 (Pin_6), J4.4 (Pin_4), R19.2, R20.2, U11.7 (~{PRE}), U11.8 (VCC), U13.3 (VDD)
- net +5V: now also C32.1, C33.1
- net 5V_EN: now also R16.2, U11.5 (Q)
- net CAN LISTEN H: now also U5.7 (CANH), U8.7 (CANH), J1.4 (Pin_4), R15.2
- net CAN LISTEN L: now also U5.6 (CANL), U8.6 (CANL), J1.5 (Pin_5), R15.1
- net GND: now also R11.2, U12.4 (GND), U3.5 (SHDN), U5.5 (SHDN), C1.1, C17.2, C18.2, C19.2, C2.1, C20.2, C21.2, C22.2, C23.2, C24.2, C25.2, C26.2, C27.2, C28.2, C29.2, C30.2, C31.2, C32.2, C33.2, C34.2, C5.1, C6.1, J1.6 (Pin_6), J2.5 (Pin_5), J3.7 (Pin_7), J4.5 (Pin_5), J5.5 (Pin_5), R14.2, R16.1, R17.1, R18.1, U11.4 (GND), U13.1 (GND), U14.2 (GND), Y4.2, Y4.4, Y5.2, Y5.4
- net ING12V+: now also D9.2 (A), J1.7 (Pin_7)
- net NRF_UART_RX: now also U2.27 (P1.00); no longer U2.35 (P0.09)
- net NRF_UART_TX: now also U2.26 (P0.22); no longer U2.36 (P0.10)
- net OBD2 CAN H: now also U3.7 (CANH), U6.7 (CANH), J1.3 (Pin_3), R21.2
- net OBD2 CAN L: now also U3.6 (CANL), U6.6 (CANL), J1.2 (Pin_2), R21.1
- net at F1.2: now also J1.1 (Pin_1)
- net NRF_SCK: now reaches U4.10 (SCK)
- net NRF_SCK: now also U2.20 (P0.19), U7.10 (SCK), J3.5 (Pin_5)
- net NRF_MOSI: now reaches U4.11 (SDI)
- net NRF_MOSI: now also U2.19 (P0.21), U7.11 (SDI), J3.4 (Pin_4)
- net NRF_MISO: now reaches U4.12 (SDO)
- net NRF_MISO: now also U2.18 (P0.23), U7.12 (SDO), J3.3 (Pin_3)
- net NRF_CS1_CAN1: now reaches U4.13 (~{CS})
- net NRF_CS1_CAN1: now also U2.15 (P0.07), R19.1
- net NRF_CAN1_INT: now reaches U4.4 (~{INT})
- net NRF_CAN1_INT: now also U2.3 (P1.10)
- net at U4.5 (OSC2): now also C1.2, Y4.3
- net at U4.6 (OSC1): now also C2.2, Y4.1
- net NRF_I2C_IRQ: now reaches U2.10 (P0.30)
- net NRF_I2C_IRQ: now also J2.1 (Pin_1)
- net NRF_SPI_CS: now reaches U2.11 (P0.31)
- net NRF_SPI_CS: now also J3.2 (Pin_2)
- net NRF_UART2_TX: now reaches U2.12 (P0.04)
- net NRF_UART2_TX: now also J4.2 (Pin_2)
- net NRF_UART2_RX: now reaches U2.13 (P0.05)
- net NRF_UART2_RX: now also J4.3 (Pin_3)
- net NRF_SDA: now reaches U2.16 (P1.09)
- net NRF_SDA: now also J2.3 (Pin_3)
- net NRF_SCL: now reaches U2.17 (P0.12)
- net NRF_SCL: now also J2.2 (Pin_2)
- net NRF_CS3_EINK: now reaches U2.2 (P1.11)
- net NRF_CS2_CAN2: now reaches U2.21 (P0.18)
- net NRF_CS2_CAN2: now also U7.13 (~{CS}), R20.1
- net NRF_UART2_IRQ: now reaches U2.28 (P1.03)
- net NRF_UART2_IRQ: now also J4.1 (Pin_1)
- net NRF_PWR_STATE: now reaches U2.29 (P1.01)
- net NRF_PWR_STATE: now also R18.2, U11.2 (D)
- net NRF_PWR_CLK: now reaches U2.30 (P1.02)
- net NRF_PWR_CLK: now also R17.2, U11.1 (CLK)
- net NRF_SPI_IRQ: now reaches U2.33 (P1.04)
- net NRF_SPI_IRQ: now also J3.1 (Pin_1)
- net NRF_CAN2_INT: now reaches U2.4 (P1.13)
- net NRF_CAN2_INT: now also U7.4 (~{INT})
- net NRF_CAN1_SHDN: now reaches U2.5 (P1.15)
- net NRF_CAN1_SHDN: now also U6.5 (SHDN)
- net NRF_ING12V+: now reaches U2.6 (P0.03)
- net NRF_ING12V+: now also C17.1, R13.2, R14.1
- net NRF_EINK_DC: now reaches U2.7 (P0.02)
- net NRF_CAN2_SHDN: now reaches U2.8 (P0.28)
- net NRF_CAN2_SHDN: now also U8.5 (SHDN)
- net NRF_RST: now reaches U2.9 (P0.29)
- net at RD1.2: now also C34.1
- net at U7.5 (OSC2): now also C5.2, Y5.3
- net at U7.6 (OSC1): now also C6.2, Y5.1
- net UART0_RX renamed LYRA_UART0_RX
- net LYRA_UART0_RX: now also U14.6 (1Y)
- net UART0_TX renamed LYRA_UART0_TX
- net LYRA_UART0_TX: now also U14.3 (2A)
- new net: D9.1 (K), R13.1
- new net: U11.6 (~{CLR}), U13.2 (~{RESET})
- new net LYRA_EXT_UART0_RX: J5.3 (Pin_3), U14.4 (2Y)
- new net LYRA_EXT_UART0_TX: J5.2 (Pin_2), U14.1 (1A)
Other:
- moved on the sheet: U2, U3, U4, U5, U6, U7, U8, U9

Commit message: update pcb
Parts:
- removed C19, C21, C25, C29: 10uF/50V-X5R(X7R)_1206, Capacitor_SMD:C_1206_3216Metric_Pad1.33x1.80mm_HandSolder, symbol ETH3:C_small_PG
- removed C24: 100nF/50V-X7R_0805, Capacitor_SMD:C_0805_2012Metric_Pad1.18x1.45mm_HandSolder, symbol ETH3:C_small_PG
- C23: value 10uF/50V-X5R(X7R)_1206 -> 100nF/50V-X7R_0805; footprint Capacitor_SMD:C_1206_3216Metric_Pad1.33x1.80mm_HandSolder -> Capacitor_SMD:C_0805_2012Metric_Pad1.18x1.45mm_HandSolder; Wartość wyśw. 10uF -> 100nF
Connections:
- net LYRA_UART1_TX: now also U1.27 (RMIO24_/_GPIO1_B1); no longer U1.7 (RMIO2_/_GPIO0_A2)
- net OBD2 CAN H: now also J1.2 (Pin_2); no longer J1.3 (Pin_3)
- net OBD2 CAN L: now also J1.3 (Pin_3); no longer J1.2 (Pin_2)

Commit message: pcb + pins update
Connections:
- net LYRA_UART1_RX: now also U1.26 (RMIO12_/_GPIO0_B4); no longer U1.32 (RMIO14_/_GPIO0_B6)
Changed lines of the file:
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@@
+	(wire
+		(pts
+			(xy 93.98 68.58) (xy 100.33 68.58)
+		)
+		(stroke
+			(width 0)
+			(type default)
+		)
+	)
 	(wire
 		(pts
@@
 		(pts
 			(xy 38.1 172.72) (xy 30.48 172.72)
-		)
-		(stroke
-			(width 0)
-			(type default)
-		)
-	)
-	(wire
-		(pts
-			(xy 93.98 76.2) (xy 100.33 76.2)
 		)
 		(stroke
@@
 		)
 	)
-	(label "LYRA_UART1_RX"
-		(at 100.33 76.2 0)
-		(effects
-			(font
-				(size 1 1)
-			)
-			(justify left bottom)
-		)
-	)
 	(label "OBD2 CAN H"
 		(at 39.37 160.02 0)
@@
 		)
 	)
+	(label "LYRA_UART1_RX"
+		(at 100.33 68.58 0)
+		(effects
+			(font
+				(size 1 1)
+			)
+			(justify left bottom)
+		)
+	)
