File: pcb/LUCKFOX-LYRA-ZEROW/LUCKFOX-LYRA-ZEROW.kicad_sch (KiCad schematic)
At the start: 73 parts, among them J1 Conn_01x07, J2 Conn_01x05, J3 Conn_01x07, J4 Conn_01x05, J5 Conn_01x05, U1 Luckfox_Lyra_Zero_W, U10 RAA211403, U11 SN74LVC1G74DCUT, U12 74LVC2G66, U13 TPS3839G33DBZT, U14 74AUP2G34GW,125, U2 CORE52840, U3 MAX3051, U4 MCP2518FD-xQBB, U5 MAX3051, U6 MAX3051, U7 MCP2518FD-xQBB, U8 MAX3051, U9 74AUP2G34GW,125, Y4 Crystal_GND24_Small, Y5 Crystal_GND24_Small

Commit message: fix mcp on pcb
Parts:
- added C19, C21, C7, C8: 22pF, Capacitor_SMD:C_0805_2012Metric, symbol Device:C_Small
- added R22, R23: (150k/1%_0805), Resistor_SMD:R_0805_2012Metric_Pad1.20x1.40mm_HandSolder, symbol ETH3:R_small_PG
- added U15, U16: MCP2518FDT-E/SL, MCP2518FD:SOIC-14_L8.7-W3.9-P1.27-LS6.0-BL, symbol MCP2518FD:MCP2518FDT-E_SL
- added Y6, Y7: Crystal_GND24_Small, Crystal:Crystal_SMD_3225-4Pin_3.2x2.5mm, symbol Device:Crystal_GND24_Small
Connections:
- net +3V3: now also R22.2, R23.2, U15.14 (VDD), U16.14 (VDD)
- net GND: now also C19.1, C21.1, C7.1, C8.1, U15.7 (VSS), U16.7 (VSS), Y6.2, Y6.4, Y7.2, Y7.4
- net NRF_CAN1_INT: now also U16.4 (~{INT})
- net NRF_CAN2_INT: now also U15.4 (~{INT})
- net NRF_CS1_CAN1: now also R22.1, U16.13 (nCS)
- net NRF_CS2_CAN2: now also R23.1, U15.13 (nCS)
- net NRF_MISO: now also U15.12 (SDO), U16.12 (SDO)
- net NRF_MOSI: now also U15.11 (SDI), U16.11 (SDI)
- net NRF_SCK: now also U15.10 (SCK), U16.10 (SCK)
- net at U6.1 (TXD): now also U16.1 (TXCAN); no longer U4.1 (TXCAN)
- net at U6.4 (RXD): now also U16.2 (RXCAN); no longer U4.2 (RXCAN)
- new net: C7.2, U16.5 (OSC2), Y6.3
- new net: C21.2, U15.6 (OSC1), Y7.1
- new net: C19.2, U15.5 (OSC2), Y7.3
- new net: C8.2, U16.6 (OSC1), Y6.1

Commit message: more pcb work
Parts:
- removed C1, C2, C5, C6: 22pF, Capacitor_SMD:C_0805_2012Metric, symbol Device:C_Small
- removed J3: Conn_01x07, Connector_JST:JST_GH_SM07B-GHS-TB_1x07-1MP_P1.25mm_Horizontal, symbol Connector_Generic:Conn_01x07
- removed R19, R20: (150k/1%_0805), Resistor_SMD:R_0805_2012Metric_Pad1.20x1.40mm_HandSolder, symbol ETH3:R_small_PG
- removed U4, U7: MCP2518FD-xQBB, Package_SO:SOIC-14_3.9x8.7mm_P1.27mm, symbol Interface_CAN_LIN:MCP2518FD-xQBB
- removed Y4, Y5: Crystal_GND24_Small, Crystal:Crystal_SMD_3225-4Pin_3.2x2.5mm, symbol Device:Crystal_GND24_Small
- added J6: Conn_01x08, Connector_JST:JST_GH_SM08B-GHS-TB_1x08-1MP_P1.25mm_Horizontal, symbol Connector_Generic:Conn_01x08
Connections:
- net +3V3: now also J6.7 (Pin_7)
- net GND: now also J6.8 (Pin_8)
- net NRF_MISO: now also J6.4 (Pin_4)
- net NRF_MOSI: now also J6.5 (Pin_5)
- net NRF_SCK: now also J6.6 (Pin_6)
- net NRF_SPI_CS: now also J6.3 (Pin_3)
- net NRF_SPI_IRQ: now also J6.2 (Pin_2)
- net NRF_SPI_RST: now reaches U2.34 (P1.06)
- net NRF_SPI_RST: now also J6.1 (Pin_1)
- net at U8.1 (TXD): now also U15.1 (TXCAN)
- net at U8.4 (RXD): now also U15.2 (RXCAN)
Other:
- moved on the sheet: U8

Commit message: more pcb work
Connections:
- net +5V: now also J5.1 (Pin_1)
Changed lines of the file:
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@@
+	)
+	(symbol
+		(lib_id "power:+5V")
+		(at 191.77 21.59 90)
+		(unit 1)
+		(body_style 1)
+		(exclude_from_sim no)
+		(in_bom yes)
+		(on_board yes)
+		(in_pos_files yes)
+		(dnp no)
+		(fields_autoplaced yes)
+		(property "Reference" "#PWR023"
+			(at 195.58 21.59 0)
+			(hide yes)
+			(show_name no)
+			(do_not_autoplace no)
+			(effects
+				(font
+					(size 1.27 1.27)
+				)
+			)
+		)
+		(property "Value" "+5V"
+			(at 187.96 21.5899 90)
+			(show_name no)
+			(do_not_autoplace no)
+			(effects
+				(font
+					(size 1.27 1.27)
+				)
+				(justify left)
+			)
+		)
+		(property "Footprint" ""
+			(at 191.77 21.59 0)
+			(hide yes)
+			(show_name no)
+			(do_not_autoplace no)
+			(effects
+				(font
+					(size 1.27 1.27)
+				)
+			)
+		)
+		(property "Datasheet" ""
+			(at 191.77 21.59 0)
+			(hide yes)
+			(show_name no)
+			(do_not_autoplace no)
+			(effects
+				(font
+					(size 1.27 1.27)
+				)
+			)
+		)
+		(property "Description" "Power symbol creates a global label with name \"+5V\""
+			(at 191.77 21.59 0)
+			(hide yes)
+			(show_name no)
+			(do_not_autoplace no)
+			(effects
+				(font
+					(size 1.27 1.27)
+				)
+			)
+		)
+		(pin "1"
+		)
+		(instances
+			(project "LUCKFOX-LYRA-ZEROW"
+				(path "/01a1a023-e48c-458b-aa28-b9cd6c31a0a1"
+					(reference "#PWR023")
+					(unit 1)
+				)
+			)
+		)
 	)
 	(symbol

Commit message: fix pcb mirror
Connections:
- net CAN0_RX: now also U1.8 (RMIO22_/_GPIO0_C6); no longer U1.37 (RMIO28_/_GPIO1_C3)
- net CAN0_TX: now also U1.7 (RMIO2_/_GPIO0_A2); no longer U1.33 (RMIO27_/_GPIO1_C2)
- net CAN1_RX: now also U1.10 (RMIO23_/_GPIO0_C7); no longer U1.31 (RMIO26_/_GPIO1_B3)
- net CAN1_TX: now also U1.12 (RMIO14_/_GPIO0_B6); no longer U1.29 (RMIO25_/_GPIO1_B2)
- net LYRA_SPI1_MISO: now also U1.18 (RMIO12_/_GPIO0_B4); no longer U1.22 (RMIO11_/_GPIO0_B3)
- net LYRA_SPI1_MOSI: now also U1.22 (RMIO11_/_GPIO0_B3); no longer U1.18 (RMIO12_/_GPIO0_B4)
- net LYRA_SPI1_SCLK: now also U1.19 (RMIO6_/_GPIO0_A6); no longer U1.23 (RMIO8_/_GPIO0_B0)
- net LYRA_UART0_RX: now also U1.24 (RMIO10_/_GPIO0_B2); no longer U1.36 (RMIO29_/_GPIO1_D1)
- net LYRA_UART0_TX: now also U1.23 (RMIO8_/_GPIO0_B0); no longer U1.38 (RMIO17_/_GPIO0_C1)
- net LYRA_UART1_RX: now also U1.16 (RMIO13_/_GPIO0_B5); no longer U1.26 (RMIO9_/_GPIO0_B1)
- net LYRA_UART1_TX: now also U1.15 (RMIO5_/_GPIO0_A5); no longer U1.27 (RMIO24_/_GPIO1_B1)
Changed lines of the file:
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@@
 	(wire
 		(pts
+			(xy 39.37 45.72) (xy 45.72 45.72)
+		)
+		(stroke
+			(width 0)
+			(type default)
+		)
+	)
+	(wire
+		(pts
+			(xy 39.37 55.88) (xy 45.72 55.88)
+		)
+		(stroke
+			(width 0)
+			(type default)
+		)
+	)
+	(wire
+		(pts
 			(xy 492.76 113.03) (xy 487.68 113.03)
 		)
@@
 	(wire
 		(pts
+			(xy 93.98 66.04) (xy 99.06 66.04)
+		)
+		(stroke
+			(width 0)
+			(type default)
+		)
+	)
+	(wire
+		(pts
 			(xy 208.28 55.88) (xy 204.47 55.88)
 		)
@@
 	(wire
 		(pts
+			(xy 93.98 48.26) (xy 97.79 48.26)
+		)
+		(stroke
+			(width 0)
+			(type default)
+		)
+	)
+	(wire
+		(pts
 			(xy 22.86 118.11) (xy 22.86 120.65)
 		)
@@
 	(wire
 		(pts
+			(xy 93.98 45.72) (xy 97.79 45.72)
+		)
+		(stroke
+			(width 0)
+			(type default)
+		)
+	)
+	(wire
+		(pts
 			(xy 208.28 45.72) (xy 204.47 45.72)
 		)
@@
 	(wire
 		(pts
+			(xy 93.98 55.88) (xy 99.06 55.88)
+		)
+		(stroke
+			(width 0)
+			(type default)
+		)
+	)
+	(wire
+		(pts
+			(xy 93.98 50.8) (xy 97.79 50.8)
+		)
+		(stroke
+			(width 0)
+			(type default)
+		)
+	)
+	(wire
+		(pts
 			(xy 524.51 88.9) (xy 528.32 88.9)
 		)
@@
 	(wire
 		(pts
+			(xy 40.64 60.96) (xy 45.72 60.96)
+		)
+		(stroke
+			(width 0)
+			(type default)
+		)
+	)
+	(wire
+		(pts
 			(xy 39.37 102.87) (xy 39.37 105.41)
 		)
@@
 		)
 	)
+	(label "LYRA_SPI1_SCLK"
+		(at 40.64 60.96 180)
+		(effects
+			(font
+				(size 1 1)
+			)
+			(justify right bottom)
+		)
+	)
 	(label "NRF_CAN2_SHDN"
 		(at 245.11 59.69 0)
@@
 	)
 	(label "CAN0_RX"
-		(at 39.37 83.82 180)
+		(at 97.79 45.72 0)
 		(effects
 			(font
 				(size 1 1)
 			)
-			(justify right bottom)
+			(justify left bottom)
 		)
 	)
@@
 		)
 	)
-	(label "LYRA_SPI1_SCLK"
-		(at 40.64 66.04 180)
-		(effects
-			(font
-				(size 1 1)
-			)
-			(justify right bottom)
-		)
-	)
 	(label "NRF_SWDIO"
 		(at 172.72 87.63 0)
@@
 	)
 	(label "LYRA_UART1_TX"
-		(at 39.37 71.12 180)
+		(at 39.37 55.88 180)
 		(effects
 			(font
@@
 	)
 	(label "CAN1_TX"
-		(at 39.37 73.66 180)
+		(at 97.79 50.8 0)
 		(effects
 			(font
 				(size 1 1)
 			)
-			(justify right bottom)
+			(justify left bottom)
 		)
 	)
@@
 	)
 	(label "LYRA_UART0_RX"
-		(at 100.33 81.28 0)
+		(at 99.06 66.04 0)
 		(effects
 			(font
@@
 	)
 	(label "LYRA_SPI1_MISO"
-		(at 99.06 63.5 0)
+		(at 99.06 58.42 0)
 		(effects
 			(font
@@
 	)
 	(label "LYRA_UART1_RX"
-		(at 100.33 68.58 0)
+		(at 99.06 55.88 0)
 		(effects
 			(font
@@
 	)
 	(label "LYRA_UART0_TX"
-		(at 100.33 83.82 0)
+		(at 40.64 66.04 180)
 		(effects
 			(font
 				(size 1 1)
 			)
-			(justify left bottom)
+			(justify right bottom)
 		)
 	)
@@
 	)
 	(label "LYRA_SPI1_MOSI"
-		(at 99.06 58.42 0)
+		(at 99.06 63.5 0)
 		(effects
 			(font
@@
 	)
 	(label "CAN1_RX"
-		(at 39.37 76.2 180)
+		(at 97.79 48.26 0)
 		(effects
 			(font
 				(size 1 1)
 			)
-			(justify right bottom)
+			(justify left bottom)
 		)
 	)
@@
 	)
 	(label "CAN0_TX"
-		(at 39.37 78.74 180)
+		(at 39.37 45.72 180)
 		(effects
 			(font

Commit message: more pcb clean up
Parts:
- added J3: Conn_01x03, Connector_JST:JST_GH_SM03B-GHS-TB_1x03-1MP_P1.25mm_Horizontal, symbol Connector_Generic:Conn_01x03
- added SW1: PCM12SMTR, PCM12SMTR:SW-SMD_PCM12SMTR, symbol PCM12SMTR:PCM12SMTR
Connections:
- net +3.3VA: now also SW1.1; no longer R11.1, U12.3, U12.7
- net GND: now also J3.3 (Pin_3), SW1.3, SW1.4
- net NRF_SWDCLK: now also J3.1 (Pin_1)
- net NRF_SWDIO: now also J3.2 (Pin_2)
- new net SWD_LYRA_EN: R11.1, SW1.2, U12.3, U12.7
