File: pcb/LUCKFOX-LYRA-ZEROW/LUCKFOX-LYRA-ZEROW.kicad_pcb (KiCad board)
At the start: 2 copper layers, 1 part, among them U1 Luckfox_Lyra_Zero_W

Commit message: slint upgrade
Parts:
- added U2: ME54BS12-nRF54L15, MinewSemi_nRF54:ME54BS12_nRF54L15, F.Cu at (145.8, 49.2)
- added U3: ME54BS01-nRF54L15, MinewSemi_nRF54:ME54BS01_nRF54L15, F.Cu at (123.0, 52.8)

Commit message: more pcb work
Parts:
- added U4: MCP2518FD-xQBB, Package_DFN_QFN:DFN-14-1EP_3x4.5mm_P0.65mm_EP1.65x4.25mm, F.Cu at (132.7, 46.8)
- added U5: MAX3051, Package_SO:SOIC-8_3.9x4.9mm_P1.27mm, F.Cu at (89.9, 62.7)
- added U6: MAX3051, Package_SO:SOIC-8_3.9x4.9mm_P1.27mm, F.Cu at (89.9, 69.3)
- added U7: MCP2518FD-xQBB, Package_DFN_QFN:DFN-14-1EP_3x4.5mm_P0.65mm_EP1.65x4.25mm, F.Cu at (97.2, 56.0)
- added U8: MAX3051, Package_SO:SOIC-8_3.9x4.9mm_P1.27mm, F.Cu at (89.9, 75.9)
- added U9: 74AUP2G34GW,125, Package_TO_SOT_SMD:SOT-363_SC-70-6_Handsoldering, F.Cu at (97.0, 61.1)
- U2: value ME54BS12-nRF54L15 -> CORE52840; footprint MinewSemi_nRF54:ME54BS12_nRF54L15 -> Core52840:BULETM-SMD_HOLYIOT-18010-NRF52840
- U3: value ME54BS01-nRF54L15 -> MAX3051; footprint MinewSemi_nRF54:ME54BS01_nRF54L15 -> Package_SO:SOIC-8_3.9x4.9mm_P1.27mm
- moved U3 33.3 mm to (89.9, 56.1)
- moved U2 24.6 mm to (121.8, 54.8)
Connections:
- U1 pad 1: unconnected-(U1-3V3-Pad1) -> +3.3VA
- U1 pad 14: unconnected-(U1-GND-Pad14) -> GND
- U1 pad 17: unconnected-(U1-3V3-Pad17) -> +3.3VA
- U1 pad 2: unconnected-(U1-5V-Pad2) -> +5V
- U1 pad 20: unconnected-(U1-GND-Pad20) -> GND
- U1 pad 25: unconnected-(U1-GND-Pad25) -> GND
- U1 pad 30: unconnected-(U1-GND-Pad30) -> GND
- U1 pad 34: unconnected-(U1-GND-Pad34) -> GND
- U1 pad 39: unconnected-(U1-GND-Pad39) -> GND
- U1 pad 4: unconnected-(U1-5V-Pad4) -> +5V
- U1 pad 6: unconnected-(U1-GND-Pad6) -> GND
- U1 pad 9: unconnected-(U1-GND-Pad9) -> GND
- U2 pad 1: unconnected-(U2-RF-Pad1) -> GND
- U2 pad 14: unconnected-(U2-P0.02-Pad14) -> +3V3
- U3 pad 2: unconnected-(U3-P1.09-Pad2) -> GND
- U3 pad 3: unconnected-(U3-P1.10-Pad3) -> +3.3VA
- U3 pad 8: unconnected-(U3-P1.06-Pad8) -> GND

Commit message: PCB LYRA work
Parts:
- added C1: 22pF, Capacitor_SMD:C_0805_2012Metric, F.Cu at (112.4, 0.66)
- added C10: 10uF/50V-X5R(X7R)_1206, Capacitor_SMD:C_1206_3216Metric_Pad1.33x1.80mm_HandSolder, F.Cu at (114.8, 58.1)
- added C11: 100nF/50V-X7R_0805, Capacitor_SMD:C_0805_2012Metric_Pad1.18x1.45mm_HandSolder, F.Cu at (117.9, 45.3)
- added C12: 10uF/16V(25V,35V,50V)-X5R(X7R)_1206, Capacitor_SMD:C_1206_3216Metric_Pad1.33x1.80mm_HandSolder, F.Cu at (107.9, 46.7)
- added C13: 10uF/16V(25V,35V,50V)-X5R(X7R)_1206, Capacitor_SMD:C_1206_3216Metric_Pad1.33x1.80mm_HandSolder, F.Cu at (107.1, 51.7)
- added C14: 10uF/16V(25V,35V,50V)-X5R(X7R)_1206, Capacitor_SMD:C_1206_3216Metric_Pad1.33x1.80mm_HandSolder, F.Cu at (105.6, 46.7)
- added C15: 10uF/50V-X5R(X7R)_1206, Capacitor_SMD:C_1206_3216Metric_Pad1.33x1.80mm_HandSolder, F.Cu at (101.7, 48.1)
- added C16: 10uF/50V-X5R(X7R)_1206, Capacitor_SMD:C_1206_3216Metric_Pad1.33x1.80mm_HandSolder, F.Cu at (94.1, 54.2)
- added C17: 100nF/50V-X7R_0805, Capacitor_SMD:C_0805_2012Metric_Pad1.18x1.45mm_HandSolder, F.Cu at (98.1, 9.69)
- added C18: 100nF/50V-X7R_0805, Capacitor_SMD:C_0805_2012Metric_Pad1.18x1.45mm_HandSolder, F.Cu at (74.0, 50.8)
- added C19: 10uF/50V-X5R(X7R)_1206, Capacitor_SMD:C_1206_3216Metric_Pad1.33x1.80mm_HandSolder, F.Cu at (72.8, 55.9)
- added C2: 22pF, Capacitor_SMD:C_0805_2012Metric, F.Cu at (112.4, 3.67)
- added C20: 100nF/50V-X7R_0805, Capacitor_SMD:C_0805_2012Metric_Pad1.18x1.45mm_HandSolder, F.Cu at (102.9, 3.67)
- added C21: 10uF/50V-X5R(X7R)_1206, Capacitor_SMD:C_1206_3216Metric_Pad1.33x1.80mm_HandSolder, F.Cu at (78.5, -18.8)
- added C22: 100nF/50V-X7R_0805, Capacitor_SMD:C_0805_2012Metric_Pad1.18x1.45mm_HandSolder, F.Cu at (102.9, 6.67)
- added C23: 10uF/50V-X5R(X7R)_1206, Capacitor_SMD:C_1206_3216Metric_Pad1.33x1.80mm_HandSolder, F.Cu at (78.5, -15.4)
- added C24: 100nF/50V-X7R_0805, Capacitor_SMD:C_0805_2012Metric_Pad1.18x1.45mm_HandSolder, F.Cu at (102.9, 9.69)
- added C25: 10uF/50V-X5R(X7R)_1206, Capacitor_SMD:C_1206_3216Metric_Pad1.33x1.80mm_HandSolder, F.Cu at (78.5, -12.1)
- added C26: 100nF/50V-X7R_0805, Capacitor_SMD:C_0805_2012Metric_Pad1.18x1.45mm_HandSolder, F.Cu at (107.7, 0.66)
- added C27: 10uF/50V-X5R(X7R)_1206, Capacitor_SMD:C_1206_3216Metric_Pad1.33x1.80mm_HandSolder, F.Cu at (78.5, -8.72)
- added C28: 100nF/50V-X7R_0805, Capacitor_SMD:C_0805_2012Metric_Pad1.18x1.45mm_HandSolder, F.Cu at (107.7, 3.67)
- added C29: 10uF/50V-X5R(X7R)_1206, Capacitor_SMD:C_1206_3216Metric_Pad1.33x1.80mm_HandSolder, F.Cu at (110.3, -9.31)
- added C3: 100nF/50V-X7R_0805, Capacitor_SMD:C_0805_2012Metric_Pad1.18x1.45mm_HandSolder, F.Cu at (98.1, 0.66)
- added C30: 100nF/50V-X7R_0805, Capacitor_SMD:C_0805_2012Metric_Pad1.18x1.45mm_HandSolder, F.Cu at (107.7, 6.67)
- added C31: 10uF/50V-X5R(X7R)_1206, Capacitor_SMD:C_1206_3216Metric_Pad1.33x1.80mm_HandSolder, F.Cu at (78.5, -5.38)
- added C32: 100nF/50V-X7R_0805, Capacitor_SMD:C_0805_2012Metric_Pad1.18x1.45mm_HandSolder, F.Cu at (107.7, 9.69)
- added C33: 10uF/50V-X5R(X7R)_1206, Capacitor_SMD:C_1206_3216Metric_Pad1.33x1.80mm_HandSolder, F.Cu at (78.5, -2.02)
- added C34: 22uF / 50V, Capacitor_SMD:C_2220_5750Metric_Pad1.97x5.40mm_HandSolder, F.Cu at (108.3, 60.1)
- added C4: 10uF/50V-X5R(X7R)_1206, Capacitor_SMD:C_1206_3216Metric_Pad1.33x1.80mm_HandSolder, F.Cu at (72.5, -22.1)
- added C5: 22pF, Capacitor_SMD:C_0805_2012Metric, F.Cu at (112.4, 6.67)
- added C6: 22pF, Capacitor_SMD:C_0805_2012Metric, F.Cu at (112.4, 9.69)
- added C9: 100nF/50V-X7R_0805, Capacitor_SMD:C_0805_2012Metric_Pad1.18x1.45mm_HandSolder, F.Cu at (114.2, 55.9)
- added D5: PMEG4020ER, Diode_SMD:D_SOD-123F, F.Cu at (118.4, 49.9)
- added D6: SKL16-AQ, Diode_SMD:D_SMA_Handsoldering, F.Cu at (99.8, 56.0)
- added D9: D, Diode_SMD:D_0805_2012Metric, F.Cu at (113.0, 12.7)
- added DL1: MPZ2012S221ATxxx (MPZ2012S331ATxxx), (BLM21PG221SH1), (CBM0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, Inductor_SMD:L_0805_2012Metric_Pad1.05x1.20mm_HandSolder, F.Cu at (48.8, 42.8)
- added DL2: SRP7028CC-220M/NRS5030T220MMGJ, Inductor_SMD:L_Bourns_SRP7028A_7.3x6.6mm, F.Cu at (112.7, 51.3)
- added DL3: 15uH, Inductor_SMD:L_Wuerth_MAPI-3015, F.Cu at (97.3, 52.2)
- added DT1: P6SMB33A, Diode_SMD:D_SMB_Handsoldering, F.Cu at (45.7, 45.6)
- added F1: Fuse_Small, Fuse:Fuseholder_Littelfuse_Nano2_154x, F.Cu at (40.6, 46.4)
- added J1: Conn_01x07, Connector_JST:JST_GH_SM07B-GHS-TB_1x07-1MP_P1.25mm_Horizontal, B.Cu at (41.1, 47.4)
- added J2: Conn_01x05, Connector_JST:JST_GH_SM05B-GHS-TB_1x05-1MP_P1.25mm_Horizontal, B.Cu at (116.2, 67.4)
- added J3: Conn_01x07, Connector_JST:JST_GH_SM07B-GHS-TB_1x07-1MP_P1.25mm_Horizontal, B.Cu at (124.3, 47.4)
- added J4: Conn_01x05, Connector_JST:JST_GH_SM05B-GHS-TB_1x05-1MP_P1.25mm_Horizontal, B.Cu at (124.3, 59.6)
- added J5: Conn_01x05, Connector_JST:JST_GH_SM05B-GHS-TB_1x05-1MP_P1.25mm_Horizontal, B.Cu at (41.1, 59.5)
- added R10: (150k/1%_0805), Resistor_SMD:R_0805_2012Metric_Pad1.20x1.40mm_HandSolder, F.Cu at (101.1, 50.2)
- added R11: 22k/1%_0805, Resistor_SMD:R_0805_2012Metric_Pad1.20x1.40mm_HandSolder, F.Cu at (95.6, -10.5)
- added R12: 1k, Resistor_SMD:R_0805_2012Metric_Pad1.20x1.40mm_HandSolder, F.Cu at (95.6, -7.58)
- added R13: 47k, Resistor_SMD:R_0805_2012Metric_Pad1.20x1.40mm_HandSolder, F.Cu at (100.3, -22.3)
- added R14: 10k, Resistor_SMD:R_0805_2012Metric_Pad1.20x1.40mm_HandSolder, F.Cu at (100.3, -19.4)
- added R15: ~, Resistor_SMD:R_0805_2012Metric_Pad1.20x1.40mm_HandSolder, F.Cu at (100.3, -16.4)
- added R16: (150k/1%_0805), Resistor_SMD:R_0805_2012Metric_Pad1.20x1.40mm_HandSolder, F.Cu at (100.3, -13.5)
- added R17: (150k/1%_0805), Resistor_SMD:R_0805_2012Metric_Pad1.20x1.40mm_HandSolder, F.Cu at (100.3, -10.5)
- added R18: (150k/1%_0805), Resistor_SMD:R_0805_2012Metric_Pad1.20x1.40mm_HandSolder, F.Cu at (100.3, -7.58)
- added R19: (150k/1%_0805), Resistor_SMD:R_0805_2012Metric_Pad1.20x1.40mm_HandSolder, F.Cu at (105.1, -22.3)
- added R20: (150k/1%_0805), Resistor_SMD:R_0805_2012Metric_Pad1.20x1.40mm_HandSolder, F.Cu at (105.1, -19.4)
- added R21: ~, Resistor_SMD:R_0805_2012Metric_Pad1.20x1.40mm_HandSolder, F.Cu at (105.1, -16.4)
- added R7: (150k/1%_0805), Resistor_SMD:R_0805_2012Metric_Pad1.20x1.40mm_HandSolder, F.Cu at (112.3, 45.8)
- added R8: 100k/1%_0805, Resistor_SMD:R_0805_2012Metric_Pad1.20x1.40mm_HandSolder, F.Cu at (110.3, 45.8)
- added R9: 22k/1%_0805, Resistor_SMD:R_0805_2012Metric_Pad1.20x1.40mm_HandSolder, F.Cu at (111.4, 42.9)
- added RD1: 0,39R MMA02040C 3907J(G,F) (0,33R MMA02040C 3307J(G,F)), (0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, Resistor_SMD:R_MiniMELF_MMA-0204, F.Cu at (108.1, 56.0)
- added S1: LMR54406FDBVR (LMR54410FDBVR), (LMR54406DBVR), (LMR54410DBV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, Package_TO_SOT_SMD:SOT-23-6_Handsoldering, F.Cu at (115.1, 45.2)
- added U10: RAA211403, RAA211403:SOT-23-5_L3.0-W1.7-P0.95-LS2.8-BL, F.Cu at (101.2, 52.7)
- added U11: SN74LVC1G74DCUT, Package_SO:VSSOP-8_2.3x2mm_P0.5mm, F.Cu at (76.3, 50.4)
- added U12: 74LVC2G66, Package_SO:TSSOP-8_3x3mm_P0.65mm, F.Cu at (75.8, 56.5)
- added U13: TPS3839G33DBZT, Package_TO_SOT_SMD:SOT-23, F.Cu at (71.3, 50.9)
- added U14: 74AUP2G34GW,125, Package_TO_SOT_SMD:SOT-363_SC-70-6_Handsoldering, F.Cu at (58.2, 48.2)
- added Y4: Crystal_GND24_Small, Crystal:Crystal_SMD_3225-4Pin_3.2x2.5mm, F.Cu at (108.1, 13.5)
- added Y5: Crystal_GND24_Small, Crystal:Crystal_SMD_3225-4Pin_3.2x2.5mm, F.Cu at (108.1, 18.0)
- U4, U7: footprint Package_DFN_QFN:DFN-14-1EP_3x4.5mm_P0.65mm_EP1.65x4.25mm -> Package_SO:SOIC-14_3.9x8.7mm_P1.27mm
- moved U6 68.5 mm to (142.8, 25.8)
- moved U9 68.5 mm to (150.0, 17.6)
- moved U7 68.5 mm to (150.1, 12.6)
- moved U8 68.5 mm to (142.8, 32.4)
- moved U4 67.2 mm to (195.2, 22.1)
- moved U3 38.6 mm to (51.9, 49.3), turned to 180 degrees
- moved U5 38.4 mm to (51.9, 57.4), turned to 180 degrees
- moved U2 36.5 mm to (85.3, 55.2), turned to 180 degrees
Connections:
- U1 pad 11: unconnected-(U1-RMIO3_/_GPIO0_A3-Pad11) -> /TOUCH_INT
- U1 pad 13: unconnected-(U1-RMIO4_/_GPIO0_A4-Pad13) -> /TOUCH_RST
- U1 pad 18: unconnected-(U1-RMIO9_/_GPIO0_B1-Pad18) -> /LYRA_SPI1_MOSI
- U1 pad 21: unconnected-(U1-RMIO7_/_GPIO0_A7-Pad21) -> /LYRA_SPI1_CS1
- U1 pad 22: unconnected-(U1-RMIO10_/_GPIO0_B2-Pad22) -> /LYRA_SPI1_MISO
- U1 pad 23: unconnected-(U1-RMIO8_/_GPIO0_B0-Pad23) -> /LYRA_SPI1_SCLK
- U1 pad 28: unconnected-(U1-RMIO13_/_GPIO0_B5-Pad28) -> /LCD_RST
- U1 pad 29: unconnected-(U1-RMIO25_/_GPIO1_B2-Pad29) -> /CAN1_TX
- U1 pad 3: unconnected-(U1-RMIO0_/_GPIO0_A0-Pad3) -> /TOUCH_SDA
- U1 pad 31: unconnected-(U1-RMIO26_/_GPIO1_B3-Pad31) -> /CAN1_RX
- U1 pad 32: unconnected-(U1-RMIO14_/_GPIO0_B6-Pad32) -> /LYRA_UART1_RX
- U1 pad 33: unconnected-(U1-RMIO27_/_GPIO1_C2-Pad33) -> /CAN0_TX
- U1 pad 36: unconnected-(U1-RMIO23_/_GPIO0_C7-Pad36) -> /LYRA_UART0_RX
- U1 pad 37: unconnected-(U1-RMIO28_/_GPIO1_C3-Pad37) -> /CAN0_RX
- U1 pad 38: unconnected-(U1-RMIO22_/_GPIO0_C6-Pad38) -> /LYRA_UART0_TX
- U1 pad 5: unconnected-(U1-RMIO1_/_GPIO0_A1-Pad5) -> /TOUCH_SCL
- U1 pad 7: unconnected-(U1-RMIO2_/_GPIO0_A2-Pad7) -> /LYRA_UART1_TX
- U2 pad 10: unconnected-(U2-P0.30-Pad10) -> /NRF_I2C_IRQ
- U2 pad 11: unconnected-(U2-P0.31-Pad11) -> /NRF_SPI_CS
- U2 pad 12: unconnected-(U2-P0.04-Pad12) -> /NRF_UART2_TX
- U2 pad 13: unconnected-(U2-P0.05-Pad13) -> /NRF_UART2_RX
- U2 pad 15: unconnected-(U2-P0.07-Pad15) -> /NRF_CS1_CAN1
- U2 pad 16: unconnected-(U2-P1.09-Pad16) -> /NRF_SDA
- U2 pad 17: unconnected-(U2-P0.12-Pad17) -> /NRF_SCL
- U2 pad 18: unconnected-(U2-P0.23-Pad18) -> /NRF_MISO
- U2 pad 19: unconnected-(U2-P0.21-Pad19) -> /NRF_MOSI
- U2 pad 2: unconnected-(U2-P1.11-Pad2) -> /NRF_CS3_EINK
- U2 pad 20: unconnected-(U2-P0.19-Pad20) -> /NRF_SCK
- U2 pad 21: unconnected-(U2-P0.18-Pad21) -> /NRF_CS2_CAN2
- U2 pad 26: unconnected-(U2-P0.22-Pad26) -> /NRF_UART_TX
- U2 pad 27: unconnected-(U2-P1.00-Pad27) -> /NRF_UART_RX
- U2 pad 28: unconnected-(U2-P1.03-Pad28) -> /NRF_UART2_IRQ
- U2 pad 29: unconnected-(U2-P1.01-Pad29) -> /NRF_PWR_STATE
- U2 pad 3: unconnected-(U2-P1.10-Pad3) -> /NRF_CAN1_INT
- U2 pad 30: unconnected-(U2-P1.02-Pad30) -> /NRF_PWR_CLK
- U2 pad 31: unconnected-(U2-SWDCLK-Pad31) -> /NRF_SWDCLK
- U2 pad 32: unconnected-(U2-SWDIO-Pad32) -> /NRF_SWDIO
- U2 pad 33: unconnected-(U2-P1.04-Pad33) -> /NRF_SPI_IRQ
- U2 pad 4: unconnected-(U2-P1.13-Pad4) -> /NRF_CAN2_INT
- U2 pad 5: unconnected-(U2-P1.15-Pad5) -> /NRF_CAN1_SHDN
- U2 pad 6: unconnected-(U2-P0.03-Pad6) -> /NRF_ING12V+
- U2 pad 7: unconnected-(U2-P0.02-Pad7) -> /NRF_EINK_DC
- U2 pad 8: unconnected-(U2-P0.28-Pad8) -> /NRF_CAN2_SHDN
- U2 pad 9: unconnected-(U2-P0.29-Pad9) -> /NRF_RST
- U3 pad 1: unconnected-(U3-TXD-Pad1) -> /CAN0_TX
- U3 pad 4: unconnected-(U3-RXD-Pad4) -> /CAN0_RX
- U3 pad 5: unconnected-(U3-SHDN-Pad5) -> GND
- U3 pad 6: unconnected-(U3-CANL-Pad6) -> /OBD2 CAN L
- U3 pad 7: unconnected-(U3-CANH-Pad7) -> /OBD2 CAN H
- U4 pad 10: unconnected-(U4-SCK-Pad10) -> /NRF_SCK
- U4 pad 11: unconnected-(U4-SDI-Pad11) -> /NRF_MOSI
- U4 pad 12: unconnected-(U4-SDO-Pad12) -> /NRF_MISO
- U4 pad 13: unconnected-(U4-~{CS}-Pad13) -> /NRF_CS1_CAN1
- U4 pad 4: unconnected-(U4-~{INT}-Pad4) -> /NRF_CAN1_INT
- U4 pad 5: unconnected-(U4-OSC2-Pad5) -> Net-(U4-OSC2)
- U4 pad 6: unconnected-(U4-OSC1-Pad6) -> Net-(U4-OSC1)
- U5 pad 1: unconnected-(U5-TXD-Pad1) -> /CAN1_TX
- U5 pad 4: unconnected-(U5-RXD-Pad4) -> /CAN1_RX
- U5 pad 5: unconnected-(U5-SHDN-Pad5) -> GND
- U5 pad 6: unconnected-(U5-CANL-Pad6) -> /CAN LISTEN L
- U5 pad 7: unconnected-(U5-CANH-Pad7) -> /CAN LISTEN H
- U6 pad 5: unconnected-(U6-SHDN-Pad5) -> /NRF_CAN1_SHDN
- U6 pad 6: unconnected-(U6-CANL-Pad6) -> /OBD2 CAN L
- U6 pad 7: unconnected-(U6-CANH-Pad7) -> /OBD2 CAN H
- U7 pad 10: unconnected-(U7-SCK-Pad10) -> /NRF_SCK
- U7 pad 11: unconnected-(U7-SDI-Pad11) -> /NRF_MOSI
- U7 pad 12: unconnected-(U7-SDO-Pad12) -> /NRF_MISO
- U7 pad 13: unconnected-(U7-~{CS}-Pad13) -> /NRF_CS2_CAN2
- U7 pad 4: unconnected-(U7-~{INT}-Pad4) -> /NRF_CAN2_INT
- U7 pad 5: unconnected-(U7-OSC2-Pad5) -> Net-(U7-OSC2)
- U7 pad 6: unconnected-(U7-OSC1-Pad6) -> Net-(U7-OSC1)
- U8 pad 5: unconnected-(U8-SHDN-Pad5) -> /NRF_CAN2_SHDN
- U8 pad 6: unconnected-(U8-CANL-Pad6) -> /CAN LISTEN L
- U8 pad 7: unconnected-(U8-CANH-Pad7) -> /CAN LISTEN H
- U9 pad 1: unconnected-(U9-1A-Pad1) -> /NRF_UART_TX
- U9 pad 2: unconnected-(U9-GND-Pad2) -> GND
- U9 pad 3: unconnected-(U9-2A-Pad3) -> /LYRA_UART1_TX
- U9 pad 4: unconnected-(U9-2Y-Pad4) -> /NRF_UART_RX
- U9 pad 5: unconnected-(U9-VCC-Pad5) -> +3.3VA
- U9 pad 6: unconnected-(U9-1Y-Pad6) -> /LYRA_UART1_RX
Routing:
- net Net-(S1-Vin): track 0.00 -> 98.3 mm, vias 0 -> 3
- net GND: track 0.00 -> 91.4 mm, vias 0 -> 21
- net +3V3: track 0.00 -> 57.6 mm, vias 0 -> 3
- net /5V_EN: track 0.00 -> 40.1 mm, vias 0 -> 2
- net +5V: track 0.00 -> 30.6 mm
- net Net-(D5-K): track 0.00 -> 29.5 mm
- net /LYRA_SPI1_MISO: track 0.00 -> 19.5 mm, vias 0 -> 1
- net /LYRA_SPI1_SCLK: track 0.00 -> 12.5 mm, vias 0 -> 1
- net +12V: track 0.00 -> 10.9 mm
- net Net-(U11-~{CLR}): track 0.00 -> 9.97 mm
- net Net-(D6-K): track 0.00 -> 9.40 mm
- net Net-(S1-FB): track 0.00 -> 8.34 mm
- net /LYRA_UART0_TX: track 0.00 -> 7.91 mm
- net Net-(C34-Pad1): track 0.00 -> 6.21 mm
- net /LYRA_UART0_RX: track 0.00 -> 5.47 mm
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- added copper zone on In1.Cu, net GND
Other:
- copper layers 2 -> 4

Commit message: update pcb
Parts:
- removed C19, C21, C25, C29: 10uF/50V-X5R(X7R)_1206, Capacitor_SMD:C_1206_3216Metric_Pad1.33x1.80mm_HandSolder
- removed C24: 100nF/50V-X7R_0805, Capacitor_SMD:C_0805_2012Metric_Pad1.18x1.45mm_HandSolder
- C23: value 10uF/50V-X5R(X7R)_1206 -> 100nF/50V-X7R_0805; footprint Capacitor_SMD:C_1206_3216Metric_Pad1.33x1.80mm_HandSolder -> Capacitor_SMD:C_0805_2012Metric_Pad1.18x1.45mm_HandSolder
- DL2: value SRP7028CC-220M/NRS5030T220MMGJ -> SRP7028CC-220M/150M
- moved U6 105.4 mm to (41.8, 55.7), turned to 90 degrees
- moved R21 92.6 mm to (46.1, 54.9), turned to -90 degrees
- moved U9 89.7 mm to (66.1, 49.4), turned to 180 degrees
- moved R15 87.3 mm to (46.1, 52.0)
- moved U8 86.5 mm to (60.0, 57.4), turned to 180 degrees
- moved R17 72.2 mm to (70.6, 55.3), turned to 90 degrees
- moved R18 70.4 mm to (68.7, 55.3), turned to 90 degrees
- moved C30 66.6 mm to (58.6, 51.6), turned to -90 degrees
- moved C31 60.1 mm to (60.8, 52.1), turned to -90 degrees
- moved U5 8.15 mm to (51.7, 49.3)
- moved U3 5.49 mm to (51.7, 54.7)
- moved U14 0.36 mm to (58.6, 48.2)
Connections:
- J1 pad 2: /OBD2 CAN L -> /OBD2 CAN H
- J1 pad 3: /OBD2 CAN H -> /OBD2 CAN L
- U1 pad 27: unconnected-(U1-RMIO24_/_GPIO1_B1-Pad27) -> /LYRA_UART1_TX
- U1 pad 7: /LYRA_UART1_TX -> unconnected-(U1-RMIO2_/_GPIO0_A2-Pad7)
Routing:
- net +3.3VA: track 0.00 -> 65.2 mm, vias 0 -> 3
- net GND: track 91.4 -> 123.7 mm, vias 21 -> 25
- net /CAN LISTEN L: track 0.00 -> 29.5 mm, vias 0 -> 3
- net /CAN LISTEN H: track 0.00 -> 22.9 mm, vias 0 -> 2
- net /OBD2 CAN H: track 0.00 -> 18.3 mm, vias 0 -> 1
- net /OBD2 CAN L: track 0.00 -> 16.5 mm, vias 0 -> 1
- net /CAN0_TX: track 0.00 -> 15.1 mm, vias 0 -> 1
- net /CAN1_TX: track 0.00 -> 14.7 mm, vias 0 -> 1
- net /NRF_PWR_STATE: track 3.77 -> 17.2 mm, vias 0 -> 2
- net /CAN0_RX: track 0.00 -> 11.1 mm
- net /CAN1_RX: track 0.00 -> 10.5 mm, vias 0 -> 1
- net /NRF_PWR_CLK: track 5.31 -> 12.4 mm, vias 0 -> 2
- net /LYRA_UART0_TX: track 7.91 -> 8.72 mm

Commit message: pcb + pins update
Connections:
- U1 pad 26: unconnected-(U1-RMIO12_/_GPIO0_B4-Pad26) -> /LYRA_UART1_RX
- U1 pad 32: /LYRA_UART1_RX -> unconnected-(U1-RMIO14_/_GPIO0_B6-Pad32)
Changed lines of the file:
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@@
 			(layers "*.Cu" "*.Mask")
 			(remove_unused_layers no)
-			(net "unconnected-(U1-RMIO12_{slash}_GPIO0_B4-Pad26)")
+			(net "/LYRA_UART1_RX")
 			(pinfunction "RMIO12_/_GPIO0_B4_26")
 			(pintype "bidirectional")
@@
 			(layers "*.Cu" "*.Mask")
 			(remove_unused_layers no)
-			(net "/LYRA_UART1_RX")
+			(net "unconnected-(U1-RMIO14_{slash}_GPIO0_B6-Pad32)")
 			(pinfunction "RMIO14_/_GPIO0_B6_32")
 			(pintype "bidirectional")

Commit message: pcb work
Parts:
- moved RD1 14.1 mm to (121.5, 60.3), turned to -90 degrees
- moved R9 9.78 mm to (109.9, 52.6), turned to -90 degrees
- moved DL2 9.30 mm to (119.6, 45.1), turned to 90 degrees
- moved C34 9.11 mm to (117.3, 58.9), turned to 90 degrees
- moved C10 7.20 mm to (118.8, 52.1), turned to -90 degrees
- moved C9 7.06 mm to (121.3, 55.9), turned to 90 degrees
- moved R7 6.85 mm to (111.8, 52.6), turned to -90 degrees
- moved C12 5.72 mm to (112.9, 43.9), turned to -90 degrees
- moved S1 5.25 mm to (115.2, 50.5), turned to 0 degrees
- moved D5 3.32 mm to (121.1, 51.8)
- moved C11 3.26 mm to (115.0, 46.8)
- moved R8 0.98 mm to (110.6, 46.7), turned to -90 degrees
Routing:
- net Net-(D5-K): track 29.5 -> 13.1 mm
- net Net-(S1-Vin): track 98.3 -> 86.6 mm, vias 3 -> 2
- net GND: track 123.7 -> 114.4 mm
- net +5V: track 30.6 -> 23.9 mm
- net Net-(S1-CB): track 1.54 -> 4.50 mm
- net Net-(C34-Pad1): track 6.21 -> 4.24 mm
- net /5V_EN: track 40.1 -> 38.1 mm
Other:
- board outline added: 89.7 x 24.1 mm

Commit message: power pcb rework
Parts:
- moved C13 7.89 mm to (104.7, 44.2)
- moved D6 7.48 mm to (101.6, 48.7)
- moved R10 6.48 mm to (97.6, 55.7), turned to 0 degrees
- moved C15 5.17 mm to (100.6, 53.1), turned to 90 degrees
- moved R8 4.37 mm to (107.1, 49.2)
- moved DL3 4.11 mm to (95.1, 48.7), turned to 180 degrees
- moved U10 3.98 mm to (97.2, 53.1), turned to -90 degrees
- moved C11 3.60 mm to (111.5, 47.0)
- moved C12 3.60 mm to (109.3, 44.2)
- moved C9 3.60 mm to (117.7, 56.2)
- moved R7 3.60 mm to (108.2, 52.9)
- moved R9 3.60 mm to (106.3, 52.9)
- moved RD1 3.60 mm to (117.9, 60.6)
- moved C10 3.60 mm to (115.2, 52.3)
- moved S1 3.60 mm to (111.6, 50.8)
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Routing:
- net Net-(S1-Vin): track 86.6 -> 116.7 mm
- net /5V_EN: track 38.1 -> 19.4 mm
- net +3V3: track 57.6 -> 41.4 mm
- net Net-(D6-K): track 9.40 -> 19.9 mm
- net Net-(J1-Pin_1): track 0.00 -> 5.42 mm, vias 0 -> 1
- net GND: track 114.4 -> 110.6 mm, vias 25 -> 28
- net +5V: track 23.9 -> 21.8 mm, vias 0 -> 2
- net Net-(S1-FB): track 8.12 -> 10.0 mm
Other:
- board size 89.7 x 24.1 mm -> 89.7 x 24.8 mm

Commit message: more pcb work
Parts:
- moved U9 1.88 mm to (67.3, 48.0)
Routing:
- net /5V_EN: track 19.4 -> 44.2 mm
- net /NRF_UART_RX: track 0.00 -> 17.3 mm, vias 0 -> 2
- net /NRF_UART_TX: track 0.00 -> 13.4 mm, vias 0 -> 2
- net /LYRA_UART1_RX: track 0.00 -> 9.98 mm
- net GND: track 110.6 -> 119.1 mm, vias 28 -> 30
- net /LYRA_UART1_TX: track 0.00 -> 2.21 mm
- net +3.3VA: track 65.2 -> 66.6 mm, vias 3 -> 4
