File: pcb/LUCKFOX-LYRA-ZEROW/LUCKFOX-LYRA-ZEROW.kicad_pcb (KiCad board)
At the start: 4 copper layers, 89.7 x 24.8 mm, 73 parts, among them J1 Conn_01x07, J2 Conn_01x05, J3 Conn_01x07, J4 Conn_01x05, J5 Conn_01x05, U1 Luckfox_Lyra_Zero_W, U10 RAA211403, U11 SN74LVC1G74DCUT, U12 74LVC2G66, U13 TPS3839G33DBZT, U14 74AUP2G34GW,125, U2 CORE52840, U3 MAX3051, U4 MCP2518FD-xQBB, U5 MAX3051, U6 MAX3051, U7 MCP2518FD-xQBB, U8 MAX3051, U9 74AUP2G34GW,125, Y4 Crystal_GND24_Small, Y5 Crystal_GND24_Small

Commit message: more pcb work
Parts:
- removed C1, C2, C5, C6: 22pF, Capacitor_SMD:C_0805_2012Metric
- removed J3: Conn_01x07, Connector_JST:JST_GH_SM07B-GHS-TB_1x07-1MP_P1.25mm_Horizontal
- removed R19, R20: (150k/1%_0805), Resistor_SMD:R_0805_2012Metric_Pad1.20x1.40mm_HandSolder
- removed U4, U7: MCP2518FD-xQBB, Package_SO:SOIC-14_3.9x8.7mm_P1.27mm
- removed Y4, Y5: Crystal_GND24_Small, Crystal:Crystal_SMD_3225-4Pin_3.2x2.5mm
- added C19: 22pF, Capacitor_SMD:C_0805_2012Metric, B.Cu at (106.7, 56.3)
- added C21: 22pF, Capacitor_SMD:C_0805_2012Metric, B.Cu at (106.7, 62.2)
- added C7: 22pF, Capacitor_SMD:C_0805_2012Metric, B.Cu at (82.6, 55.4)
- added C8: 22pF, Capacitor_SMD:C_0805_2012Metric, B.Cu at (84.1, 52.1)
- added J6: Conn_01x08, Connector_JST:JST_GH_SM08B-GHS-TB_1x08-1MP_P1.25mm_Horizontal, B.Cu at (124.3, 47.2)
- added R22: (150k/1%_0805), Resistor_SMD:R_0805_2012Metric_Pad1.20x1.40mm_HandSolder, B.Cu at (97.4, 61.7)
- added R23: (150k/1%_0805), Resistor_SMD:R_0805_2012Metric_Pad1.20x1.40mm_HandSolder, F.Cu at (94.9, 58.5)
- added U15: MCP2518FDT-E/SL, MCP2518FD:SOIC-14_L8.7-W3.9-P1.27-LS6.0-BL, F.Cu at (103.8, 59.8)
- added U16: MCP2518FDT-E/SL, MCP2518FD:SOIC-14_L8.7-W3.9-P1.27-LS6.0-BL, B.Cu at (91.1, 58.2)
- added Y6: Crystal_GND24_Small, Crystal:Crystal_SMD_3225-4Pin_3.2x2.5mm, B.Cu at (85.3, 55.2)
- added Y7: Crystal_GND24_Small, Crystal:Crystal_SMD_3225-4Pin_3.2x2.5mm, B.Cu at (107.1, 59.2)
- moved D9 70.4 mm to (49.6, 43.5), turned to 180 degrees
- moved DL1 1.50 mm to (49.9, 41.7), turned to 0 degrees
- moved J4 0.25 mm to (124.3, 59.9)
Connections:
- U2 pad 34: unconnected-(U2-P1.06-Pad34) -> /NRF_SPI_RST
Routing:
- net +3V3: track 41.4 -> 98.2 mm, vias 3 -> 6
- net Net-(U16-TXCAN): track 0.00 -> 52.0 mm, vias 0 -> 1
- net Net-(U15-RXCAN): track 0.00 -> 49.0 mm, vias 0 -> 2
- net Net-(U16-RXCAN): track 0.00 -> 45.8 mm, vias 0 -> 1
- net Net-(U15-TXCAN): track 0.00 -> 38.9 mm, vias 0 -> 2
- net /NRF_SCK: track 0.00 -> 29.9 mm, vias 0 -> 3
- net /NRF_MOSI: track 0.00 -> 28.3 mm, vias 0 -> 2
- net /NRF_CS2_CAN2: track 0.00 -> 28.2 mm, vias 0 -> 2
- net /NRF_MISO: track 0.00 -> 27.1 mm, vias 0 -> 2
- net /NRF_CS1_CAN1: track 0.00 -> 25.0 mm, vias 0 -> 1
- net GND: track 119.1 -> 140.9 mm, vias 30 -> 33
- net /NRF_CAN2_INT: track 0.00 -> 13.8 mm
- net Net-(U15-OSC1): track 0.00 -> 8.93 mm, vias 0 -> 1
- net Net-(U15-OSC2): track 0.00 -> 7.41 mm, vias 0 -> 1
- net Net-(U16-OSC2): track 0.00 -> 6.96 mm
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
Commit message: more pcb work
Parts:
- moved R13 84.6 mm to (49.8, 45.5)
- moved R14 81.2 mm to (62.9, 52.7), turned to -90 degrees
- moved R11 68.2 mm to (66.8, 51.3), turned to -90 degrees
- moved R16 67.3 mm to (120.6, 50.7), turned to 180 degrees
- moved R12 66.4 mm to (72.6, 54.7), turned to -90 degrees
- moved C17 54.3 mm to (64.9, 52.7), turned to -90 degrees
Routing:
- net /NRF_ING12V+: track 0.00 -> 44.6 mm, vias 0 -> 2
- net /LYRA_SPI1_MOSI: track 0.00 -> 20.0 mm, vias 0 -> 2
- net GND: track 140.9 -> 152.8 mm, vias 33 -> 35
- net /5V_EN: track 44.2 -> 50.9 mm, vias 2 -> 3
- net +3.3VA: track 66.6 -> 70.5 mm
- net Net-(D9-K): track 0.00 -> 2.69 mm
- net /LYRA_SPI1_MISO: track 19.5 -> 22.2 mm
- net +3V3: track 98.2 -> 99.8 mm

Commit message: more pcb work
Parts:
- moved J2 3.38 mm to (118.5, 67.4)
- moved C8 0.91 mm to (83.2, 52.1)
- moved J5 0.75 mm to (41.1, 58.7)
- moved J1 0.68 mm to (41.1, 46.7)
Connections:
- J5 pad 1: unconnected-(J5-Pin_1-Pad1) -> +5V
Routing:
- net +5V: track 21.8 -> 106.5 mm, vias 2 -> 3
- net GND: track 152.8 -> 217.9 mm, vias 35 -> 42
- net /NRF_SPI_RST: track 0.00 -> 62.6 mm, vias 0 -> 2
- net /NRF_CAN1_SHDN: track 0.00 -> 61.7 mm, vias 0 -> 2
- net /NRF_SPI_IRQ: track 0.00 -> 60.2 mm, vias 0 -> 2
- net /NRF_UART2_IRQ: track 0.00 -> 51.1 mm, vias 0 -> 4
- net /NRF_SCL: track 0.00 -> 51.0 mm, vias 0 -> 2
- net +3V3: track 99.8 -> 149.8 mm
- net /NRF_CAN2_SHDN: track 0.00 -> 48.6 mm, vias 0 -> 3
- net /NRF_SDA: track 0.00 -> 47.2 mm, vias 0 -> 1
- net /NRF_SPI_CS: track 0.00 -> 43.3 mm, vias 0 -> 1
- net /NRF_I2C_IRQ: track 0.00 -> 40.7 mm, vias 0 -> 2
- net /NRF_UART2_RX: track 0.00 -> 38.5 mm, vias 0 -> 2
- net /NRF_UART2_TX: track 0.00 -> 36.6 mm, vias 0 -> 2
- net /NRF_MISO: track 27.1 -> 62.8 mm, vias 2 -> 3
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Other:
- board size 89.7 x 24.8 mm -> 89.7 x 30.7 mm

Commit message: fix pcb mirror
Parts:
- C20, C3, C4, U1: moved to B.Cu
- moved C26 87.8 mm to (44.2, 61.2)
- moved C32 85.3 mm to (39.8, 61.2), turned to 180 degrees
- moved C23 74.4 mm to (65.5, 57.9), turned to -90 degrees
- moved C4 68.4 mm to (47.4, 41.5)
- moved C27 67.8 mm to (69.0, 58.4)
- moved C22 64.0 mm to (68.6, 60.7)
- moved C28 63.7 mm to (62.9, 49.0), turned to -90 degrees
- moved C3 62.9 mm to (51.1, 42.4), turned to 90 degrees
- moved C33 62.7 mm to (120.7, 44.2), turned to -90 degrees
- moved U1 48.3 mm to (53.6, 45.2), turned to 0 degrees
- moved C20 46.9 mm to (96.3, 50.0)
Connections:
- U1 pad 10: unconnected-(U1-RMIO23_/_GPIO0_C7-Pad10) -> /CAN1_RX
- U1 pad 12: unconnected-(U1-RMIO14_/_GPIO0_B6-Pad12) -> /CAN1_TX
- U1 pad 15: unconnected-(U1-RMIO5_/_GPIO0_A5-Pad15) -> /LYRA_UART1_TX
- U1 pad 16: unconnected-(U1-RMIO13_/_GPIO0_B5-Pad16) -> /LYRA_UART1_RX
- U1 pad 18: /LYRA_SPI1_MOSI -> /LYRA_SPI1_MISO
- U1 pad 19: unconnected-(U1-RMIO6_/_GPIO0_A6-Pad19) -> /LYRA_SPI1_SCLK
- U1 pad 22: /LYRA_SPI1_MISO -> /LYRA_SPI1_MOSI
- U1 pad 23: /LYRA_SPI1_SCLK -> /LYRA_UART0_TX
- U1 pad 24: unconnected-(U1-RMIO10_/_GPIO0_B2-Pad24) -> /LYRA_UART0_RX
- U1 pad 26: /LYRA_UART1_RX -> unconnected-(U1-RMIO9_/_GPIO0_B1-Pad26)
- U1 pad 27: /LYRA_UART1_TX -> unconnected-(U1-RMIO24_/_GPIO1_B1-Pad27)
- U1 pad 29: /CAN1_TX -> unconnected-(U1-RMIO25_/_GPIO1_B2-Pad29)
- U1 pad 31: /CAN1_RX -> unconnected-(U1-RMIO26_/_GPIO1_B3-Pad31)
- U1 pad 33: /CAN0_TX -> unconnected-(U1-RMIO27_/_GPIO1_C2-Pad33)
- U1 pad 36: /LYRA_UART0_RX -> unconnected-(U1-RMIO29_/_GPIO1_D1-Pad36)
- U1 pad 37: /CAN0_RX -> unconnected-(U1-RMIO28_/_GPIO1_C3-Pad37)
- U1 pad 38: /LYRA_UART0_TX -> unconnected-(U1-RMIO17_/_GPIO0_C1-Pad38)
- U1 pad 7: unconnected-(U1-RMIO2_/_GPIO0_A2-Pad7) -> /CAN0_TX
- U1 pad 8: unconnected-(U1-RMIO22_/_GPIO0_C6-Pad8) -> /CAN0_RX
Routing:
- net GND: track 217.9 -> 246.5 mm, vias 42 -> 44
- net /LYRA_UART0_TX: track 8.72 -> 34.7 mm, vias 0 -> 1
- net /LYRA_UART0_RX: track 5.32 -> 27.1 mm
- net +3.3VA: track 104.6 -> 87.4 mm, vias 5 -> 7
- net +5V: track 106.5 -> 123.3 mm
- net +12V: track 10.9 -> 19.7 mm, vias 0 -> 2
- net +3V3: track 149.8 -> 158.1 mm
- net /CAN0_RX: track 11.1 -> 18.3 mm
- net /LYRA_SPI1_MOSI: track 20.0 -> 15.3 mm
- net /CAN1_RX: track 10.5 -> 12.8 mm
- net /CAN1_TX: track 14.7 -> 16.9 mm
- net /LYRA_SPI1_MISO: track 22.2 -> 20.0 mm
- net /NRF_SPI_RST: track 62.6 -> 61.1 mm
- net /LYRA_UART1_TX: track 2.21 -> 3.63 mm
- net /LYRA_SPI1_SCLK: track 12.5 -> 11.5 mm
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- added copper zone on B.Cu, net GND
- added copper zone on F.Cu, net GND
- added copper zone on In2.Cu, net GND

Commit message: more pcb stuff
Parts:
- moved C32 0.61 mm to (40.4, 61.2)
Connections:
- J1 pad MP: (no net) -> GND
- J2 pad MP: (no net) -> GND
- J4 pad MP: (no net) -> GND
- J5 pad MP: (no net) -> GND
- J6 pad MP: (no net) -> GND
Routing:
- net GND: track 246.5 -> 249.5 mm
- net /CAN LISTEN H: track 25.6 -> 26.9 mm
- net +5V: track 123.3 -> 124.2 mm
Other:
- outline, holes or cut-outs redrawn

Commit message: more pcb clean up
Parts:
- added J3: Conn_01x03, Connector_JST:JST_GH_SM03B-GHS-TB_1x03-1MP_P1.25mm_Horizontal, F.Cu at (124.3, 58.6)
- added SW1: PCM12SMTR, PCM12SMTR:SW-SMD_PCM12SMTR, F.Cu at (71.8, 62.2)
- moved C22 2.99 mm to (65.6, 60.8), turned to 180 degrees
Connections:
- R11 pad 1: +3.3VA -> /SWD_LYRA_EN
- U12 pad 3: +3.3VA -> /SWD_LYRA_EN
- U12 pad 7: +3.3VA -> /SWD_LYRA_EN
Routing:
- net /NRF_SWDIO: track 4.59 -> 63.3 mm, vias 0 -> 2
- net /NRF_SWDCLK: track 3.84 -> 60.3 mm, vias 0 -> 2
- net /SWD_LYRA_EN: track 0.00 -> 24.0 mm, vias 0 -> 3
- net +3V3: track 158.1 -> 168.9 mm
- net +3.3VA: track 87.4 -> 90.6 mm
- net GND: track 249.5 -> 246.9 mm, vias 44 -> 46
- net Net-(U16-TXCAN): track 52.0 -> 54.2 mm
- net Net-(U15-RXCAN): track 49.0 -> 50.1 mm
- net /NRF_CAN2_SHDN: track 48.6 -> 49.3 mm
- net Net-(U16-RXCAN): track 45.8 -> 46.5 mm
- net /NRF_UART2_IRQ: vias 4 -> 3
Other:
- outline, holes or cut-outs redrawn

Commit message: more pcb work
Parts:
- moved U2 0.06 mm to (85.2, 55.1)
Connections:
- J1 pad MP: GND -> (no net)
- J2 pad MP: GND -> (no net)
- J4 pad MP: GND -> (no net)
- J5 pad MP: GND -> (no net)
- J6 pad MP: GND -> (no net)
Routing:
- net GND: track 246.9 -> 270.1 mm
- net /NRF_CAN1_SHDN: track 61.7 -> 59.1 mm
- net +3V3: track 168.9 -> 166.6 mm
- net /CAN LISTEN H: track 26.9 -> 26.2 mm
Other:
- outline, holes or cut-outs redrawn
